File: LightDrum/ActiveFilters_1-4.kicad_sch (KiCad schematic)
At the start: 57 parts, among them U27 LMV324, U28 LMV324, U29 LMV324

Commit message: Add docs and gerbers for REV7
Other:
- title: AUDIO FILTER CHANNELS  1 - 4 -> LightDrum
Changed lines of the file:
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@@
   (paper "A4")
   (title_block
-    (title "AUDIO FILTER CHANNELS  1 - 4")
-    (rev "REV6")
+    (title "LightDrum")
+    (rev "REV7")
     (company "Daxxn Industries")
   )
