File: LightDrum/ActiveFilters_5-8.kicad_sch (KiCad schematic)
At the start: 55 parts, among them U3 LMV324, U4 LMV324, U5 LMV324

Commit message: Add docs and gerbers for REV7
Other:
- title: AUDIO FILTER CHANNELS  5 - 8 -> LightDrum
Changed lines of the file:
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@@
   (paper "A4")
   (title_block
-    (title "AUDIO FILTER CHANNELS  5 - 8")
-    (rev "REV6")
+    (title "LightDrum")
+    (rev "REV7")
     (company "Daxxn Industries")
   )
