File: LightDrum/Audio_Amp.kicad_sch (KiCad schematic)
At the start: 14 parts, among them Q1 MMBT2222A, U6 LM358, U7 OPA1652

Commit message: Add docs and gerbers for REV7
Other:
- title: AUDIO AMPLIFIER AND BIASING -> LightDrum
Changed lines of the file:
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@@
   (paper "A4")
   (title_block
-    (title "AUDIO AMPLIFIER AND BIASING")
-    (rev "REV6")
+    (title "LightDrum")
+    (rev "REV7")
     (company "Daxxn Industries")
   )
