File: LightDrum/LED_Connector.kicad_sch (KiCad schematic)
At the start: 1 part, among them J1 LED D-SUB

Commit message: Add docs and gerbers for REV7
Other:
- title: RGB STRIP CONNECTOR -> LightDrum
Changed lines of the file:
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@@
   (paper "A4")
   (title_block
-    (title "RGB STRIP CONNECTOR")
-    (rev "REV6")
+    (title "LightDrum")
+    (rev "REV7")
     (company "Daxxn Industries")
   )
