File: LightDrum/LED_MUX.kicad_sch (KiCad schematic)
At the start: 10 parts, among them Q3 MMBT2222A, U44 MIC1555, U45 CD4017B, U46 74HC02, U47 SN74LVC1G32

Commit message: Add docs and gerbers for REV7
Other:
- company: (none) -> Daxxn Industries
- title: (none) -> LightDrum
Changed lines of the file:
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@@
 (kicad_sch (version 20211123) (generator eeschema)
   (paper "A4")
+  (title_block
+    (title "LightDrum")
+    (rev "REV7")
+    (company "Daxxn Industries")
+  )
   (junction (at 158.75 46.99) (diameter 0) (color 0 0 0 0)
   )
