File: LightDrum/Battery-Charger.kicad_sch (KiCad schematic)
At the start: 4 parts, among them U903 LTC4054ES5-4.2

Commit message: Replace with smaller case (WIP)
Parts:
- removed BAT901: 20mm COIN, Daxxn_Batteries:BatteryHolder_Keystone_3002_1x2032, symbol Device:Battery_Cell
- removed C901: 100nF, Capacitor_SMD:C_0603_1608Metric, symbol Device:C_Small
- removed R905: 1.2K, Resistor_SMD:R_0603_1608Metric, symbol Device:R_Small_US
- removed U903: LTC4054ES5-4.2, Package_TO_SOT_SMD:TSOT-23-5, symbol Battery_Management:LTC4054ES5-4.2
Changed lines of the file:
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@@
 (kicad_sch (version 20211123) (generator eeschema)
   (paper "A4")
-  (junction (at 60.96 49.53) (diameter 0) (color 0 0 0 0)
-  )
-  (junction (at 78.74 36.83) (diameter 0) (color 0 0 0 0)
-  )
-  (junction (at 46.99 49.53) (diameter 0) (color 0 0 0 0)
-  )
-  (wire (pts (xy 78.74 49.53) (xy 60.96 49.53))
-    (stroke (width 0) (type default) (color 0 0 0 0))
-  )
-  (wire (pts (xy 60.96 29.21) (xy 60.96 26.67))
-    (stroke (width 0) (type default) (color 0 0 0 0))
-  )
-  (wire (pts (xy 78.74 46.99) (xy 78.74 49.53))
-    (stroke (width 0) (type default) (color 0 0 0 0))
-  )
-  (wire (pts (xy 46.99 36.83) (xy 50.8 36.83))
-    (stroke (width 0) (type default) (color 0 0 0 0))
-  )
-  (wire (pts (xy 78.74 36.83) (xy 82.55 36.83))
-    (stroke (width 0) (type default) (color 0 0 0 0))
-  )
-  (wire (pts (xy 50.8 39.37) (xy 46.99 39.37))
-    (stroke (width 0) (type default) (color 0 0 0 0))
-  )
-  (wire (pts (xy 46.99 49.53) (xy 60.96 49.53))
-    (stroke (width 0) (type default) (color 0 0 0 0))
-  )
-  (wire (pts (xy 60.96 49.53) (xy 60.96 46.99))
-    (stroke (width 0) (type default) (color 0 0 0 0))
-  )
-  (wire (pts (xy 78.74 36.83) (xy 71.12 36.83))
-    (stroke (width 0) (type default) (color 0 0 0 0))
-  )
-  (wire (pts (xy 46.99 49.53) (xy 46.99 50.8))
-    (stroke (width 0) (type default) (color 0 0 0 0))
-  )
-  (wire (pts (xy 46.99 39.37) (xy 46.99 40.64))
-    (stroke (width 0) (type default) (color 0 0 0 0))
-  )
-  (wire (pts (xy 78.74 39.37) (xy 78.74 36.83))
-    (stroke (width 0) (type default) (color 0 0 0 0))
-  )
-  (wire (pts (xy 46.99 45.72) (xy 46.99 49.53))
-    (stroke (width 0) (type default) (color 0 0 0 0))
-  )
-  (hierarchical_label "VBAT" (shape output) (at 82.55 36.83 0)
-    (effects (font (size 1.27 1.27)) (justify left))
-  )
-  (hierarchical_label "CHARGE-STATUS" (shape output) (at 46.99 36.83 180)
-    (effects (font (size 1.27 1.27)) (justify right))
-  )
-  (symbol (lib_id "Device:R_Small_US") (at 46.99 43.18 0) (unit 1)
-    (in_bom yes) (on_board yes)
-    (property "Reference" "R905" (id 0) (at 47.752 42.672 0)
-      (effects (font (size 1.27 1.27)) (justify left))
-    )
-    (property "Value" "1.2K" (id 1) (at 47.752 44.196 0)
-      (effects (font (size 1.27 1.27)) (justify left))
-    )
-    (property "Footprint" "Resistor_SMD:R_0603_1608Metric" (id 2) (at 46.99 43.18 0)
-      (effects (font (size 1.27 1.27)) hide)
-    )
-    (property "Datasheet" "~" (id 3) (at 46.99 43.18 0)
-      (effects (font (size 1.27 1.27)) hide)
-    )
-    (pin "1")
-    (pin "2")
-  )
-  (symbol (lib_id "Battery_Management:LTC4054ES5-4.2") (at 60.96 36.83 0) (unit 1)
-    (in_bom yes) (on_board yes)
-    (property "Reference" "U903" (id 0) (at 55.118 30.226 0))
-    (property "Value" "LTC4054ES5-4.2" (id 1) (at 62.484 30.226 0)
-      (effects (font (size 1.27 1.27)) (justify left))
-    )
-    (property "Footprint" "Package_TO_SOT_SMD:TSOT-23-5" (id 2) (at 60.96 49.53 0)
-      (effects (font (size 1.27 1.27)) hide)
-    )
-    (property "Datasheet" "https://www.analog.com/media/en/technical-documentation/data-sheets/405442xf.pdf" (id 3) (at 60.96 39.37 0)
-      (effects (font (size 1.27 1.27)) hide)
-    )
-    (pin "1")
-    (pin "2")
-    (pin "3")
-    (pin "4")
-    (pin "5")
-  )
-  (symbol (lib_id "power:GND") (at 46.99 50.8 0) (unit 1)
-    (in_bom yes) (on_board yes)
-    (property "Reference" "#PWR0910" (id 0) (at 46.99 57.15 0)
-      (effects (font (size 1.27 1.27)) hide)
-    )
-    (property "Value" "GND" (id 1) (at 46.99 54.61 0))
-    (property "Footprint" "" (id 2) (at 46.99 50.8 0)
-      (effects (font (size 1.27 1.27)) hide)
-    )
-    (property "Datasheet" "" (id 3) (at 46.99 50.8 0)
-      (effects (font (size 1.27 1.27)) hide)
-    )
-    (pin "1")
-  )
-  (symbol (lib_id "power:VCC") (at 81.28 17.78 0) (unit 1)
-    (in_bom yes) (on_board yes)
-    (property "Reference" "#PWR0907" (id 0) (at 81.28 21.59 0)
-      (effects (font (size 1.27 1.27)) hide)
-    )
-    (property "Value" "VCC" (id 1) (at 81.28 13.97 0))
-    (property "Footprint" "" (id 2) (at 81.28 17.78 0)
-      (effects (font (size 1.27 1.27)) hide)
-    )
-    (property "Datasheet" "" (id 3) (at 81.28 17.78 0)
-      (effects (font (size 1.27 1.27)) hide)
-    )
-    (pin "1")
-  )
-  (symbol (lib_id "Device:Battery_Cell") (at 78.74 44.45 0) (unit 1)
-    (in_bom yes) (on_board yes)
-    (property "Reference" "BAT901" (id 0) (at 81.28 41.91 0)
-      (effects (font (size 1.27 1.27)) (justify left))
-    )
-    (property "Value" "20mm COIN" (id 1) (at 81.28 44.45 0)
-      (effects (font (size 1.27 1.27)) (justify left))
-    )
-    (property "Footprint" "Daxxn_Batteries:BatteryHolder_Keystone_3002_1x2032" (id 2) (at 78.74 42.926 90)
-      (effects (font (size 1.27 1.27)) hide)
-    )
-    (property "Datasheet" "~" (id 3) (at 78.74 42.926 90)
-      (effects (font (size 1.27 1.27)) hide)
-    )
-    (pin "1")
-    (pin "2")
-  )
-  (symbol (lib_id "power:VCC") (at 60.96 26.67 0) (unit 1)
-    (in_bom yes) (on_board yes)
-    (property "Reference" "#PWR0909" (id 0) (at 60.96 30.48 0)
-      (effects (font (size 1.27 1.27)) hide)
-    )
-    (property "Value" "VCC" (id 1) (at 60.96 22.86 0))
-    (property "Footprint" "" (id 2) (at 60.96 26.67 0)
-      (effects (font (size 1.27 1.27)) hide)
-    )
-    (property "Datasheet" "" (id 3) (at 60.96 26.67 0)
-      (effects (font (size 1.27 1.27)) hide)
-    )
-    (pin "1")
-  )
-  (symbol (lib_id "Device:C_Small") (at 81.28 20.32 0) (unit 1)
-    (in_bom yes) (on_board yes)
-    (property "Reference" "C901" (id 0) (at 81.534 18.542 0)
-      (effects (font (size 1.27 1.27)) (justify left))
-    )
-    (property "Value" "100nF" (id 1) (at 81.534 22.352 0)
-      (effects (font (size 1.27 1.27)) (justify left))
-    )
-    (property "Footprint" "Capacitor_SMD:C_0603_1608Metric" (id 2) (at 81.28 20.32 0)
-      (effects (font (size 1.27 1.27)) hide)
-    )
-    (property "Datasheet" "~" (id 3) (at 81.28 20.32 0)
-      (effects (font (size 1.27 1.27)) hide)
-    )
-    (pin "1")
-    (pin "2")
-  )
-  (symbol (lib_id "power:GND") (at 81.28 22.86 0) (unit 1)
-    (in_bom yes) (on_board yes)
-    (property "Reference" "#PWR0908" (id 0) (at 81.28 29.21 0)
-      (effects (font (size 1.27 1.27)) hide)
-    )
-    (property "Value" "GND" (id 1) (at 81.28 26.67 0))
-    (property "Footprint" "" (id 2) (at 81.28 22.86 0)
-      (effects (font (size 1.27 1.27)) hide)
-    )
-    (property "Datasheet" "" (id 3) (at 81.28 22.86 0)
-      (effects (font (size 1.27 1.27)) hide)
-    )
-    (pin "1")
-  )
 )
