File: LightDrum/LightDrum.kicad_pcb (KiCad board)
At the start: 4 copper layers, 151 x 83 mm, 209 parts, among them J102 JTAG, J1201 0525593652, J1203 PWR-CONN, J201 XLR3, J202 SJ-43515RS-SMT-TR, J601 LED D-SUB, J901 STD BARREL JACK, J902 STD BARREL JACK, K901 ALQ112, K902 ALQ112, Q101 RQ5A030AP, SW101 SW_SPDT, U1001 AP3401, U1002 LM22673-SOIC, U101 STM32F103VEH6, U102 24LC04, U301 PCA9634_TSSOP20, U302 SQ2310ES_SOT23, U303 SQ2310ES_SOT23, U304 SQ2310ES_SOT23, U305 SQ2310ES_SOT23, U306 SQ2310ES_SOT23, U307 SQ2310ES_SOT23, U308 SQ2310ES_SOT23, U309 SQ2310ES_SOT23, U401 PCA9634_TSSOP20, U402 SQ2310ES_SOT23, U403 SQ2310ES_SOT23, U404 SQ2310ES_SOT23, U405 SQ2310ES_SOT23, U406 SQ2310ES_SOT23, U407 SQ2310ES_SOT23, U408 SQ2310ES_SOT23, U409 SQ2310ES_SOT23, U501 PCA9634_TSSOP20, U502 SQ2310ES_SOT23, U503 SQ2310ES_SOT23, U504 SQ2310ES_SOT23, U505 SQ2310ES_SOT23, U506 SQ2310ES_SOT23, U507 SQ2310ES_SOT23, U508 SQ2310ES_SOT23, U509 SQ2310ES_SOT23, U701 INA4181 A2, U702 INA4181 A2, U901 74HC2G08, U902 SSM3K361R_SOT23F, U903 LTC4054ES5-4.2, Y101 8MHz, Y102 32.768KHz

Commit message: Replace with smaller case (WIP)
Parts:
- removed BAT901: 20mm COIN, Daxxn_Batteries:BatteryHolder_Keystone_3002_1x2032
- removed C901: 100nF, Capacitor_SMD:C_0603_1608Metric
- removed R905: 1.2K, Resistor_SMD:R_0603_1608Metric
- removed the REF** at (109.0, 75.0)
- removed U903: LTC4054ES5-4.2, Package_TO_SOT_SMD:TSOT-23-5
- added REF**: LeMotech_Black_ENC-115x90, Daxxn_Enclosures:LeMotech_Black_ENC-115x90, F.Cu at (0.00, 0.00)
- C1015, C1016, C1017, D201, D202, D901, R213, R214: moved to B.Cu
- moved H4 164.7 mm to (39.5, -35.0)
- moved C1017 162.8 mm to (29.0, 33.5), turned to -90 degrees
- moved C1015 161.9 mm to (32.0, 34.0), turned to -90 degrees
- moved D901 160.8 mm to (14.6, 16.7), turned to 0 degrees
- moved R301 160.3 mm to (19.5, -19.5)
- moved R302 160.3 mm to (21.5, -9.50)
- moved R303 160.3 mm to (23.5, -19.5)
- moved R304 160.3 mm to (25.5, -9.50)
- moved R305 160.3 mm to (19.0, -22.5)
- moved R306 160.3 mm to (21.0, -12.5)
- moved R307 160.3 mm to (23.0, -22.5)
- moved R308 160.3 mm to (25.0, -12.5)
- moved R309 160.3 mm to (11.5, -19.5)
- moved R310 160.3 mm to (13.5, -9.50)
- moved R311 160.3 mm to (15.5, -19.5)
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Connections:
- J1201 pad 14: GND -> /Interface Connectors/CHARGE-STATUS
- J1201 pad 23: GND -> /Interface Connectors/VBAT
- J1201 pad 24: GND -> VCC
- J1201 pad 33: VCC -> VDD
- U101 pad A2: /MENU-LEFT -> unconnected-(U101-PadA2)
- U101 pad B2: /MENU-DOWN -> unconnected-(U101-PadB2)
- U101 pad B5: /AUDIO-RELAY -> unconnected-(U101-PadB5)
- U101 pad B6: /DIAG-DEBUG -> unconnected-(U101-PadB6)
- U101 pad B7: unconnected-(U101-PadB7) -> /DIAG-DEBUG
- U101 pad B8: unconnected-(U101-PadB8) -> /ENC1-B
- U101 pad B9: unconnected-(U101-PadB9) -> /MENU-DOWN
- U101 pad C2: /MENU-ACT -> unconnected-(U101-PadC2)
- U101 pad C3: /MENU-BACK -> unconnected-(U101-PadC3)
- U101 pad C9: unconnected-(U101-PadC9) -> /MENU-LEFT
- U101 pad D2: /MENU-UP -> unconnected-(U101-PadD2)
- U101 pad D3: /MENU-RIGHT -> unconnected-(U101-PadD3)
- U101 pad E2: /ENC1-B -> unconnected-(U101-PadE2)
- U101 pad E8: unconnected-(U101-PadE8) -> /MENU-UP
- U101 pad E9: unconnected-(U101-PadE9) -> /MENU-BACK
- U101 pad F8: unconnected-(U101-PadF8) -> /MENU-ACT
- U101 pad F9: unconnected-(U101-PadF9) -> /MENU-RIGHT
- U101 pad K8: /PWM-OE -> unconnected-(U101-PadK8)
- U101 pad K9: unconnected-(U101-PadK9) -> /PWM-OE
Routing:
- net /RGB_Control/RGB Control 3/LED4-R: track 0.00 -> 11.6 mm
- net /RGB_Control/RGB Control 3/LED4-G: track 0.00 -> 11.6 mm
- net /RGB_Control/RGB Control 3/LED4-B: track 0.00 -> 11.6 mm
- net /RGB_Control/RGB Control 3/LED3-B: track 0.00 -> 11.6 mm
- net /RGB_Control/RGB Control 2/LED3-R: track 0.00 -> 11.6 mm
- net /RGB_Control/RGB Control 2/LED3-G: track 0.00 -> 11.6 mm
- net /RGB_Control/RGB Control 2/LED2-R: track 0.00 -> 11.6 mm
- net /RGB_Control/RGB Control 2/LED2-B: track 0.00 -> 11.6 mm
- net /RGB_Control/RGB Control 1/LED2-G: track 0.00 -> 11.6 mm
- net /RGB_Control/RGB Control 1/LED1-R: track 0.00 -> 11.6 mm
- net /RGB_Control/RGB Control 1/LED1-G: track 0.00 -> 11.6 mm
- net /RGB_Control/RGB Control 1/LED1-B: track 0.00 -> 11.6 mm
- net Net-(C114-Pad1): track 0.00 -> 8.85 mm
- net /RGB_Control/Strip Connector/STRIP8-PWR: track 0.00 -> 7.65 mm
- net /RGB_Control/Strip Connector/STRIP5-PWR: track 0.00 -> 7.54 mm
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- added copper zone on B.Cu, net Net-(F901-Pad1)
Other:
- board size 151 x 83 mm -> 108 x 83 mm
