File: LightDrum/LightDrum.kicad_pcb (KiCad board)
At the start: 4 copper layers, 108 x 81.5 mm, 307 parts, among them J1 SWD CONN, J2 0525593652, J4 PWR-CONN, J5 DIN-4-SH, J6 XLR3, J7 SJ-63073E, J8 LED D-SUB, Q1 NTMFS5C430NLT1G, Q10 PMXB43UNEZ, Q11 PMXB43UNEZ, Q12 PMXB43UNEZ, Q13 PMXB43UNEZ, Q14 PMXB43UNEZ, Q15 PMXB43UNEZ, Q16 PMXB43UNEZ, Q17 PMXB43UNEZ, Q18 PMXB43UNEZ, Q19 PMXB43UNEZ, Q2 NX6008NBKWX, Q20 PMXB43UNEZ, Q21 PMXB43UNEZ, Q22 PMXB43UNEZ, Q23 PMXB43UNEZ, Q24 PMXB43UNEZ, Q25 PMXB43UNEZ, Q26 PMXB43UNEZ, Q27 PMXB43UNEZ, Q3 NX6008NBKWX, Q4 PMXB43UNEZ, Q5 PMXB43UNEZ, Q6 PMXB43UNEZ, Q7 PMXB43UNEZ, Q8 PMXB43UNEZ, Q9 PMXB43UNEZ, SW1 BOOT0, T1 NET-TIE, T10 NET-TIE, T11 NET-TIE, T12 NET-TIE, T13 NET-TIE, T14 NET-TIE, T15 NET-TIE, T16 NET-TIE, T2 NET-TIE, T3 NET-TIE, T4 NET-TIE, T5 NET-TIE, T6 NET-TIE, T7 NET-TIE, T8 NET-TIE, T9 NET-TIE, U1 STR485, U10 PCA9634_TSSOP20, U11 PCA9634_TSSOP20, U2 AP3401, U3 LM22673-5V, U4 TPS7A94, U5 INA4181 A2, U6 INA4181 A2, U7 SLG55021, U8 PCM1821, U9 PCA9634_TSSOP20, Y1 16MHz, Y2 32.768KHz

Commit message: Continuing layout
Parts:
- U8: footprint Daxxn_Packages:TI-WQFN-RTE-20-3x3mm-P0.5mm-EP1_1.4mm -> Daxxn_Packages:TI-WQFN-RTE_(CUSTOM)-20-3x3mm-P0.5mm-EP1_1.4mm
- moved J4 44.8 mm to (101.0, 85.0)
- moved J2 12.1 mm to (63.0, 96.0)
- moved TP4 7.89 mm to (58.0, 66.4)
- moved R24 5.10 mm to (83.6, 68.7)
- moved C7 5.10 mm to (84.3, 76.4)
- moved R3 5.10 mm to (82.2, 75.8)
- moved C3 5.10 mm to (76.9, 89.7)
- moved C37 5.10 mm to (77.0, 68.5)
- moved C38 5.10 mm to (85.5, 67.7)
- moved C39 5.10 mm to (84.2, 67.2)
- moved C4 5.10 mm to (69.7, 75.3)
- moved C40 5.10 mm to (95.5, 78.4)
- moved C41 5.10 mm to (84.9, 70.0)
- moved C42 5.10 mm to (79.5, 90.8)
- moved C43 5.10 mm to (86.2, 77.3)
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Routing:
- net VCC: track 33.1 -> 74.7 mm, vias 4 -> 7
- net /VDD-PG: track 3.72 -> 18.8 mm, vias 0 -> 2
- net VDD: track 8.69 -> 17.8 mm, vias 4 -> 10
- net /AUDIO INPUTS/JACK+: track 0.00 -> 4.25 mm
- net /AUDIO INPUTS/JACK-: track 0.00 -> 4.22 mm
- net GND: track 5.70 -> 9.70 mm, vias 26 -> 37
- net Net-(U8-SDOUT): track 0.00 -> 2.09 mm
- net Net-(Q23-G): track 0.00 -> 1.98 mm
- net Net-(Q4-G): track 0.00 -> 1.97 mm
- net Net-(Q21-G): track 0.00 -> 1.97 mm
- net Net-(Q18-G): track 0.00 -> 1.97 mm
- net Net-(Q15-G): track 0.00 -> 1.97 mm
- net Net-(Q20-G): track 0.00 -> 1.97 mm
- net Net-(Q7-G): track 0.00 -> 1.97 mm
- net Net-(Q25-G): track 0.00 -> 1.97 mm
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- added copper zone on F.Cu, net /AUDIO INPUTS/XLR+
- added copper zone on B.Cu, net Net-(C66-Pad1)
