File: LightDrum/RGB_Control-2.kicad_sch (KiCad schematic)
At the start: 25 parts, among them U17 PCA9634_TSSOP20, U18 SQ2310ES_SOT23, U19 SQ2310ES_SOT23, U20 SQ2310ES_SOT23, U21 SQ2310ES_SOT23, U22 SQ2310ES_SOT23, U23 SQ2310ES_SOT23, U24 SQ2310ES_SOT23, U25 SQ2310ES_SOT23

Commit message: Add docs and gerbers for REV7
Other:
- title: RGB STRIP CONTROLLER 2 -> LightDrum
Changed lines of the file:
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@@
   (paper "A4")
   (title_block
-    (title "RGB STRIP CONTROLLER 2")
-    (rev "REV6")
+    (title "LightDrum")
+    (rev "REV7")
     (company "Daxxn Industries")
   )

Commit message: First pass over schematic (WIP)
Parts:
- R55, R57, R59, R61, R63, R65, R67, R69: value ${GATE-RES} -> 100
- R56, R58, R60, R62, R64, R66, R68, R70: value ${P-RES} -> 10K
Changed lines of the file:
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@@
   (title_block
     (title "LightDrum")
-    (rev "REV7")
+    (rev "REV8")
     (company "Daxxn Industries")
   )
@@
       (effects (font (size 1.27 1.27)) hide)
     )
-    (property "Datasheet" "C:\\Users\\Daxxn\\Documents\\Electrical\\Datasheets\\SQ2310ES.pdf" (id 3) (at 101.6 36.83 0)
+    (property "Datasheet" "%LOCAL_DATASHEETS%\\SQ2310ES.pdf" (id 3) (at 101.6 36.83 0)
       (effects (font (size 1.27 1.27)) hide)
     )
@@
       (effects (font (size 1.27 1.27)) (justify right))
     )
-    (property "Value" "${P-RES}" (id 1) (at 171.45 54.356 0)
+    (property "Value" "10K" (id 1) (at 171.45 54.356 0)
       (effects (font (size 1.27 1.27)) (justify right))
     )
@@
       (effects (font (size 1.27 1.27)) hide)
     )
-    (property "Datasheet" "C:\\Users\\Daxxn\\Documents\\Electrical\\Datasheets\\SQ2310ES.pdf" (id 3) (at 165.1 60.96 0)
+    (property "Datasheet" "%LOCAL_DATASHEETS%\\SQ2310ES.pdf" (id 3) (at 165.1 60.96 0)
       (effects (font (size 1.27 1.27)) hide)
     )
@@
       (effects (font (size 1.27 1.27)) hide)
     )
-    (property "Datasheet" "C:\\Users\\Daxxn\\Documents\\Electrical\\Datasheets\\PCA9634.pdf" (id 3) (at 45.72 13.97 0)
+    (property "Datasheet" "%LOCAL_DATASHEETS%\\PCA9634.pdf" (id 3) (at 45.72 13.97 0)
       (effects (font (size 1.27 1.27)) hide)
     )
@@
       (effects (font (size 1.27 1.27)) hide)
     )
-    (property "Datasheet" "C:\\Users\\Daxxn\\Documents\\Electrical\\Datasheets\\SQ2310ES.pdf" (id 3) (at 177.8 36.83 0)
+    (property "Datasheet" "%LOCAL_DATASHEETS%\\SQ2310ES.pdf" (id 3) (at 177.8 36.83 0)
       (effects (font (size 1.27 1.27)) hide)
     )
@@
       (effects (font (size 1.27 1.27)) hide)
     )
-    (property "Datasheet" "C:\\Users\\Daxxn\\Documents\\Electrical\\Datasheets\\SQ2310ES.pdf" (id 3) (at 139.7 60.96 0)
+    (property "Datasheet" "%LOCAL_DATASHEETS%\\SQ2310ES.pdf" (id 3) (at 139.7 60.96 0)
       (effects (font (size 1.27 1.27)) hide)
     )
@@
       (effects (font (size 1.27 1.27)) (justify right))
     )
-    (property "Value" "${P-RES}" (id 1) (at 184.15 78.486 0)
+    (property "Value" "10K" (id 1) (at 184.15 78.486 0)
       (effects (font (size 1.27 1.27)) (justify right))
     )
@@
       (effects (font (size 1.27 1.27)) (justify right))
     )
-    (property "Value" "${GATE-RES}" (id 1) (at 171.45 46.736 0)
+    (property "Value" "100" (id 1) (at 171.45 46.99 0)
       (effects (font (size 1.27 1.27)) (justify right))
     )
@@
       (effects (font (size 1.27 1.27)) (justify right))
     )
-    (property "Value" "${GATE-RES}" (id 1) (at 158.75 70.866 0)
+    (property "Value" "100" (id 1) (at 158.75 70.866 0)
       (effects (font (size 1.27 1.27)) (justify right))
     )
@@
       (effects (font (size 1.27 1.27)) (justify right))
     )
-    (property "Value" "${P-RES}" (id 1) (at 107.95 78.486 0)
+    (property "Value" "10K" (id 1) (at 107.95 78.486 0)
       (effects (font (size 1.27 1.27)) (justify right))
     )
@@
       (effects (font (size 1.27 1.27)) (justify right))
     )
-    (property "Value" "${GATE-RES}" (id 1) (at 146.05 46.736 0)
+    (property "Value" "100" (id 1) (at 146.05 46.736 0)
       (effects (font (size 1.27 1.27)) (justify right))
     )
@@
       (effects (font (size 1.27 1.27)) (justify right))
     )
-    (property "Value" "${GATE-RES}" (id 1) (at 133.35 70.866 0)
+    (property "Value" "100" (id 1) (at 133.35 70.866 0)
       (effects (font (size 1.27 1.27)) (justify right))
     )
@@
       (effects (font (size 1.27 1.27)) hide)
     )
-    (property "Datasheet" "C:\\Users\\Daxxn\\Documents\\Electrical\\Datasheets\\SQ2310ES.pdf" (id 3) (at 114.3 60.96 0)
+    (property "Datasheet" "%LOCAL_DATASHEETS%\\SQ2310ES.pdf" (id 3) (at 114.3 60.96 0)
       (effects (font (size 1.27 1.27)) hide)
     )
@@
       (effects (font (size 1.27 1.27)) (justify right))
     )
-    (property "Value" "${GATE-RES}" (id 1) (at 120.65 46.736 0)
+    (property "Value" "100" (id 1) (at 120.65 46.736 0)
       (effects (font (size 1.27 1.27)) (justify right))
     )
@@
       (effects (font (size 1.27 1.27)) hide)
     )
-    (property "Datasheet" "C:\\Users\\Daxxn\\Documents\\Electrical\\Datasheets\\SQ2310ES.pdf" (id 3) (at 127 36.83 0)
+    (property "Datasheet" "%LOCAL_DATASHEETS%\\SQ2310ES.pdf" (id 3) (at 127 36.83 0)
       (effects (font (size 1.27 1.27)) hide)
     )
@@
       (effects (font (size 1.27 1.27)) (justify right))
     )
-    (property "Value" "${P-RES}" (id 1) (at 146.05 54.356 0)
+    (property "Value" "10K" (id 1) (at 146.05 54.356 0)
       (effects (font (size 1.27 1.27)) (justify right))
     )
@@
       (effects (font (size 1.27 1.27)) (justify right))
     )
-    (property "Value" "${P-RES}" (id 1) (at 133.35 78.486 0)
+    (property "Value" "10K" (id 1) (at 133.35 78.486 0)
       (effects (font (size 1.27 1.27)) (justify right))
     )
@@
       (effects (font (size 1.27 1.27)) (justify right))
     )
-    (property "Value" "${GATE-RES}" (id 1) (at 95.25 46.736 0)
+    (property "Value" "100" (id 1) (at 95.25 46.736 0)
       (effects (font (size 1.27 1.27)) (justify right))
     )
@@
       (effects (font (size 1.27 1.27)) (justify right))
     )
-    (property "Value" "${GATE-RES}" (id 1) (at 107.95 70.866 0)
+    (property "Value" "100" (id 1) (at 107.95 70.866 0)
       (effects (font (size 1.27 1.27)) (justify right))
     )
@@
       (effects (font (size 1.27 1.27)) (justify right))
     )
-    (property "Value" "${P-RES}" (id 1) (at 158.75 78.486 0)
+    (property "Value" "10K" (id 1) (at 158.75 78.486 0)
       (effects (font (size 1.27 1.27)) (justify right))
     )
@@
       (effects (font (size 1.27 1.27)) hide)
     )
-    (property "Datasheet" "C:\\Users\\Daxxn\\Documents\\Electrical\\Datasheets\\SQ2310ES.pdf" (id 3) (at 190.5 60.96 0)
+    (property "Datasheet" "%LOCAL_DATASHEETS%\\SQ2310ES.pdf" (id 3) (at 190.5 60.96 0)
       (effects (font (size 1.27 1.27)) hide)
     )
@@
       (effects (font (size 1.27 1.27)) (justify right))
     )
-    (property "Value" "${P-RES}" (id 1) (at 120.65 54.356 0)
+    (property "Value" "10K" (id 1) (at 120.65 54.356 0)
       (effects (font (size 1.27 1.27)) (justify right))
     )
@@
       (effects (font (size 1.27 1.27)) (justify right))
     )
-    (property "Value" "${GATE-RES}" (id 1) (at 184.15 70.866 0)
+    (property "Value" "100" (id 1) (at 184.15 70.866 0)
       (effects (font (size 1.27 1.27)) (justify right))
     )
@@
       (effects (font (size 1.27 1.27)) hide)
     )
-    (property "Datasheet" "C:\\Users\\Daxxn\\Documents\\Electrical\\Datasheets\\SQ2310ES.pdf" (id 3) (at 152.4 36.83 0)
+    (property "Datasheet" "%LOCAL_DATASHEETS%\\SQ2310ES.pdf" (id 3) (at 152.4 36.83 0)
       (effects (font (size 1.27 1.27)) hide)
     )
@@
       (effects (font (size 1.27 1.27)) (justify right))
     )
-    (property "Value" "${P-RES}" (id 1) (at 95.25 54.356 0)
-      (effects (font (size 1.27 1.27)) (justify right))
-    )
+    (property "Value" "10K" (id 1) (at 95.25 54.356 0)
+      (effects (font (size 1.27 1.27)) (justify right))
+    )

Commit message: General component placement
Parts:
- U401: renamed from U17; PartNumber (none) -> 0806-0003
- U402: renamed from U18; PartNumber (none) -> 0703-0001
- U403: renamed from U20; PartNumber (none) -> 0703-0001
- U404: renamed from U22; PartNumber (none) -> 0703-0001
- U405: renamed from U24; PartNumber (none) -> 0703-0001
- U406: renamed from U19; PartNumber (none) -> 0703-0001
- U407: renamed from U21; PartNumber (none) -> 0703-0001
- U408: renamed from U23; PartNumber (none) -> 0703-0001
- U409: renamed from U25; PartNumber (none) -> 0703-0001
- renumbered R55 to R401, R59 to R402, R63 to R403, R67 to R404, R56 to R405, R60 to R406, R64 to R407, R68 to R408, R57 to R409, R61 to R410, R65 to R411, R69 to R412, R58 to R413, R62 to R414, R66 to R415, R70 to R416

Commit message: Simplify analog power supply and add some routing
Connections:
- net LED2-B-SIG: now also U401.12 (LED5); no longer U401.9 (LED3)
- net LED2-R-SIG: now also U401.14 (LED7); no longer U401.7 (LED1)
- net LED3-G-SIG: now also U401.6 (LED0); no longer U401.11 (LED4)
- net LED3-R-SIG: now also U401.8 (LED2); no longer U401.14 (LED7)
- net LED6-B-SIG: now also U401.11 (LED4); no longer U401.8 (LED2)
- net LED6-R-SIG: now also U401.13 (LED6); no longer U401.6 (LED0)
- net LED7-G-SIG: now also U401.7 (LED1); no longer U401.12 (LED5)
- net LED7-R-SIG: now also U401.9 (LED3); no longer U401.13 (LED6)
- net VCC renamed VDD
Changed lines of the file:
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@@
     (effects (font (size 1.27 1.27)) (justify left bottom))
   )
-  (label "LED3-G-SIG" (at 55.88 41.91 0)
+  (label "LED3-G-SIG" (at 55.88 31.75 0)
     (effects (font (size 1.27 1.27)) (justify left bottom))
   )
@@
     (effects (font (size 1.27 1.27)) (justify left bottom))
   )
-  (label "LED6-B-SIG" (at 55.88 36.83 0)
+  (label "LED6-B-SIG" (at 55.88 41.91 0)
     (effects (font (size 1.27 1.27)) (justify left bottom))
   )
@@
     (effects (font (size 1.27 1.27)) (justify left bottom))
   )
-  (label "LED7-G-SIG" (at 55.88 44.45 0)
-    (effects (font (size 1.27 1.27)) (justify left bottom))
-  )
-  (label "LED3-R-SIG" (at 55.88 49.53 0)
-    (effects (font (size 1.27 1.27)) (justify left bottom))
-  )
-  (label "LED6-R-SIG" (at 55.88 31.75 0)
+  (label "LED7-G-SIG" (at 55.88 34.29 0)
+    (effects (font (size 1.27 1.27)) (justify left bottom))
+  )
+  (label "LED3-R-SIG" (at 55.88 36.83 0)
+    (effects (font (size 1.27 1.27)) (justify left bottom))
+  )
+  (label "LED6-R-SIG" (at 55.88 46.99 0)
     (effects (font (size 1.27 1.27)) (justify left bottom))
   )
@@
     (effects (font (size 1.27 1.27)) (justify left bottom))
   )
-  (label "LED2-B-SIG" (at 55.88 39.37 0)
-    (effects (font (size 1.27 1.27)) (justify left bottom))
-  )
-  (label "LED7-R-SIG" (at 55.88 46.99 0)
+  (label "LED2-B-SIG" (at 55.88 44.45 0)
+    (effects (font (size 1.27 1.27)) (justify left bottom))
+  )
+  (label "LED7-R-SIG" (at 55.88 39.37 0)
     (effects (font (size 1.27 1.27)) (justify left bottom))
   )
@@
     (effects (font (size 1.27 1.27)) (justify left bottom))
   )
-  (label "LED2-R-SIG" (at 55.88 34.29 0)
+  (label "LED2-R-SIG" (at 55.88 49.53 0)
     (effects (font (size 1.27 1.27)) (justify left bottom))
   )
@@
   (hierarchical_label "LED3-R" (shape output) (at 140.97 68.58 0)
     (effects (font (size 1.27 1.27)) (justify left))
-  )
-  (symbol (lib_id "power:VCC") (at 45.72 22.86 0) (unit 1)
-    (in_bom yes) (on_board yes)
-    (property "Reference" "#PWR0401" (id 0) (at 45.72 26.67 0)
-      (effects (font (size 1.27 1.27)) hide)
-    )
-    (property "Value" "VCC" (id 1) (at 45.72 19.05 0))
-    (property "Footprint" "" (id 2) (at 45.72 22.86 0)
-      (effects (font (size 1.27 1.27)) hide)
-    )
-    (property "Datasheet" "" (id 3) (at 45.72 22.86 0)
-      (effects (font (size 1.27 1.27)) hide)
-    )
-    (pin "1")
   )
   (symbol (lib_id "Daxxn_Transistors:SQ2310ES_SOT23") (at 100.33 49.53 0) (unit 1)
@@
     (pin "3")
   )
+  (symbol (lib_id "power:VDD") (at 45.72 22.86 0) (unit 1)
+    (in_bom yes) (on_board yes)
+    (property "Reference" "#PWR0127" (id 0) (at 45.72 26.67 0)
+      (effects (font (size 1.27 1.27)) hide)
+    )
+    (property "Value" "VDD" (id 1) (at 45.72 19.05 0))
+    (property "Footprint" "" (id 2) (at 45.72 22.86 0)
+      (effects (font (size 1.27 1.27)) hide)
+    )
+    (property "Datasheet" "" (id 3) (at 45.72 22.86 0)
+      (effects (font (size 1.27 1.27)) hide)
+    )
+    (pin "1")
+  )
   (symbol (lib_id "power:GND") (at 190.5 82.55 0) (unit 1)
     (in_bom yes) (on_board yes)
@@
     (pin "2")
   )
-  (symbol (lib_id "power:VCC") (at 20.32 39.37 0) (unit 1)
-    (in_bom yes) (on_board yes)
-    (property "Reference" "#PWR0402" (id 0) (at 20.32 43.18 0)
-      (effects (font (size 1.27 1.27)) hide)
-    )
-    (property "Value" "VCC" (id 1) (at 20.32 35.56 0))
+  (symbol (lib_id "Device:R_Small_US") (at 109.22 77.47 0) (unit 1)
+    (in_bom yes) (on_board yes)
+    (property "Reference" "R413" (id 0) (at 107.95 76.708 0)
+      (effects (font (size 1.27 1.27)) (justify right))
+    )
+    (property "Value" "10K" (id 1) (at 107.95 78.486 0)
+      (effects (font (size 1.27 1.27)) (justify right))
+    )
+    (property "Footprint" "Resistor_SMD:R_0805_2012Metric" (id 2) (at 109.22 77.47 0)
+      (effects (font (size 1.27 1.27)) hide)
+    )
+    (property "Datasheet" "~" (id 3) (at 109.22 77.47 0)
+      (effects (font (size 1.27 1.27)) hide)
+    )
+    (pin "1")
+    (pin "2")
+  )
+  (symbol (lib_id "Device:R_Small_US") (at 147.32 45.72 0) (unit 1)
+    (in_bom yes) (on_board yes)
+    (property "Reference" "R403" (id 0) (at 146.05 44.958 0)
+      (effects (font (size 1.27 1.27)) (justify right))
+    )
+    (property "Value" "100" (id 1) (at 146.05 46.736 0)
+      (effects (font (size 1.27 1.27)) (justify right))
+    )
+    (property "Footprint" "Resistor_SMD:R_0805_2012Metric" (id 2) (at 147.32 45.72 0)
+      (effects (font (size 1.27 1.27)) hide)
+    )
+    (property "Datasheet" "~" (id 3) (at 147.32 45.72 0)
+      (effects (font (size 1.27 1.27)) hide)
+    )
+    (pin "1")
+    (pin "2")
+  )
+  (symbol (lib_id "Device:R_Small_US") (at 134.62 69.85 0) (unit 1)
+    (in_bom yes) (on_board yes)
+    (property "Reference" "R410" (id 0) (at 133.35 69.088 0)
+      (effects (font (size 1.27 1.27)) (justify right))
+    )
+    (property "Value" "100" (id 1) (at 133.35 70.866 0)
+      (effects (font (size 1.27 1.27)) (justify right))
+    )
+    (property "Footprint" "Resistor_SMD:R_0805_2012Metric" (id 2) (at 134.62 69.85 0)
+      (effects (font (size 1.27 1.27)) hide)
+    )
+    (property "Datasheet" "~" (id 3) (at 134.62 69.85 0)
+      (effects (font (size 1.27 1.27)) hide)
+    )
+    (pin "1")
+    (pin "2")
+  )
+  (symbol (lib_name "SQ2310ES_SOT23_6") (lib_id "Daxxn_Transistors:SQ2310ES_SOT23") (at 113.03 73.66 0) (unit 1)
+    (in_bom yes) (on_board yes)
+    (property "Reference" "U406" (id 0) (at 115.57 72.39 0)
+      (effects (font (size 1.27 1.27)) (justify left))
+    )
+    (property "Value" "SQ2310ES_SOT23" (id 1) (at 115.57 74.93 0)
+      (effects (font (size 0.85 0.85)) (justify left))
+    )
+    (property "Footprint" "Package_TO_SOT_SMD:SOT-23" (id 2) (at 114.3 58.42 0)
+      (effects (font (size 1.27 1.27)) hide)
+    )
+    (property "Datasheet" "%LOCAL_DATASHEETS%\\SQ2310ES.pdf" (id 3) (at 114.3 60.96 0)
+      (effects (font (size 1.27 1.27)) hide)
+    )
+    (property "PartNumber" "0703-0001" (id 4) (at 115.57 69.85 0)
+      (effects (font (size 1.27 1.27)) (justify left))
+    )
+    (pin "1")
+    (pin "2")
+    (pin "3")
+  )
+  (symbol (lib_id "power:VDD") (at 20.32 39.37 0) (unit 1)
+    (in_bom yes) (on_board yes)
+    (property "Reference" "#PWR0128" (id 0) (at 20.32 43.18 0)
+      (effects (font (size 1.27 1.27)) hide)
+    )
+    (property "Value" "VDD" (id 1) (at 20.32 35.56 0))
     (property "Footprint" "" (id 2) (at 20.32 39.37 0)
       (effects (font (size 1.27 1.27)) hide)
@@
     (pin "1")
   )
-  (symbol (lib_id "Device:R_Small_US") (at 109.22 77.47 0) (unit 1)
-    (in_bom yes) (on_board yes)
-    (property "Reference" "R413" (id 0) (at 107.95 76.708 0)
-      (effects (font (size 1.27 1.27)) (justify right))
-    )
-    (property "Value" "10K" (id 1) (at 107.95 78.486 0)
-      (effects (font (size 1.27 1.27)) (justify right))
-    )
-    (property "Footprint" "Resistor_SMD:R_0805_2012Metric" (id 2) (at 109.22 77.47 0)
-      (effects (font (size 1.27 1.27)) hide)
-    )
-    (property "Datasheet" "~" (id 3) (at 109.22 77.47 0)
-      (effects (font (size 1.27 1.27)) hide)
-    )
-    (pin "1")
-    (pin "2")
-  )
-  (symbol (lib_id "Device:R_Small_US") (at 147.32 45.72 0) (unit 1)
-    (in_bom yes) (on_board yes)
-    (property "Reference" "R403" (id 0) (at 146.05 44.958 0)
-      (effects (font (size 1.27 1.27)) (justify right))
-    )
-    (property "Value" "100" (id 1) (at 146.05 46.736 0)
-      (effects (font (size 1.27 1.27)) (justify right))
-    )
-    (property "Footprint" "Resistor_SMD:R_0805_2012Metric" (id 2) (at 147.32 45.72 0)
-      (effects (font (size 1.27 1.27)) hide)
-    )
-    (property "Datasheet" "~" (id 3) (at 147.32 45.72 0)
-      (effects (font (size 1.27 1.27)) hide)
-    )
-    (pin "1")
-    (pin "2")
-  )
-  (symbol (lib_id "Device:R_Small_US") (at 134.62 69.85 0) (unit 1)
-    (in_bom yes) (on_board yes)
-    (property "Reference" "R410" (id 0) (at 133.35 69.088 0)
-      (effects (font (size 1.27 1.27)) (justify right))
-    )
-    (property "Value" "100" (id 1) (at 133.35 70.866 0)
-      (effects (font (size 1.27 1.27)) (justify right))
-    )
-    (property "Footprint" "Resistor_SMD:R_0805_2012Metric" (id 2) (at 134.62 69.85 0)
-      (effects (font (size 1.27 1.27)) hide)
-    )
-    (property "Datasheet" "~" (id 3) (at 134.62 69.85 0)
-      (effects (font (size 1.27 1.27)) hide)
-    )
-    (pin "1")
-    (pin "2")
-  )
-  (symbol (lib_name "SQ2310ES_SOT23_6") (lib_id "Daxxn_Transistors:SQ2310ES_SOT23") (at 113.03 73.66 0) (unit 1)
-    (in_bom yes) (on_board yes)
-    (property "Reference" "U406" (id 0) (at 115.57 72.39 0)
-      (effects (font (size 1.27 1.27)) (justify left))
-    )
-    (property "Value" "SQ2310ES_SOT23" (id 1) (at 115.57 74.93 0)
-      (effects (font (size 0.85 0.85)) (justify left))
-    )
-    (property "Footprint" "Package_TO_SOT_SMD:SOT-23" (id 2) (at 114.3 58.42 0)
-      (effects (font (size 1.27 1.27)) hide)
-    )
-    (property "Datasheet" "%LOCAL_DATASHEETS%\\SQ2310ES.pdf" (id 3) (at 114.3 60.96 0)
-      (effects (font (size 1.27 1.27)) hide)
-    )
-    (property "PartNumber" "0703-0001" (id 4) (at 115.57 69.85 0)
-      (effects (font (size 1.27 1.27)) (justify left))
-    )
-    (pin "1")
-    (pin "2")
-    (pin "3")
-  )
   (symbol (lib_id "Device:R_Small_US") (at 121.92 45.72 0) (unit 1)
