File: LightDrum/RGB_Control-3.kicad_sch (KiCad schematic)
At the start: 25 parts, among them Q501 PMXB43UNEZ, Q502 PMXB43UNEZ, Q503 PMXB43UNEZ, Q504 PMXB43UNEZ, Q505 PMXB43UNEZ, Q506 PMXB43UNEZ, Q507 PMXB43UNEZ, Q508 PMXB43UNEZ, U501 PCA9634_TSSOP20

Commit message: Lock REV8 Layout and send to PCB MNF
Parts:
- R501, R502, R503, R504, R505, R506, R507, R508, R509, R510, R511, R512, R513, R514, R515, R516: footprint Resistor_SMD:R_0603_1608Metric -> Resistor_SMD:R_0402_1005Metric
Changed lines of the file:
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@@
       (effects (font (size 1.27 1.27)) (justify right))
     )
-    (property "Footprint" "Resistor_SMD:R_0603_1608Metric" (id 2) (at 134.62 73.66 0)
+    (property "Footprint" "Resistor_SMD:R_0402_1005Metric" (id 2) (at 134.62 73.66 0)
       (effects (font (size 1.27 1.27)) hide)
     )
@@
       (effects (font (size 1.27 1.27)) (justify right))
     )
-    (property "Footprint" "Resistor_SMD:R_0603_1608Metric" (id 2) (at 172.72 49.53 0)
+    (property "Footprint" "Resistor_SMD:R_0402_1005Metric" (id 2) (at 172.72 49.53 0)
       (effects (font (size 1.27 1.27)) hide)
     )
@@
       (effects (font (size 1.27 1.27)) (justify right))
     )
-    (property "Footprint" "Resistor_SMD:R_0603_1608Metric" (id 2) (at 134.62 81.28 0)
+    (property "Footprint" "Resistor_SMD:R_0402_1005Metric" (id 2) (at 134.62 81.28 0)
       (effects (font (size 1.27 1.27)) hide)
     )
@@
       (effects (font (size 1.27 1.27)) (justify right))
     )
-    (property "Footprint" "Resistor_SMD:R_0603_1608Metric" (id 2) (at 96.52 57.15 0)
+    (property "Footprint" "Resistor_SMD:R_0402_1005Metric" (id 2) (at 96.52 57.15 0)
       (effects (font (size 1.27 1.27)) hide)
     )
@@
       (effects (font (size 1.27 1.27)) (justify right))
     )
-    (property "Footprint" "Resistor_SMD:R_0603_1608Metric" (id 2) (at 185.42 81.28 0)
+    (property "Footprint" "Resistor_SMD:R_0402_1005Metric" (id 2) (at 185.42 81.28 0)
       (effects (font (size 1.27 1.27)) hide)
     )
@@
       (effects (font (size 1.27 1.27)) (justify right))
     )
-    (property "Footprint" "Resistor_SMD:R_0603_1608Metric" (id 2) (at 121.92 57.15 0)
+    (property "Footprint" "Resistor_SMD:R_0402_1005Metric" (id 2) (at 121.92 57.15 0)
       (effects (font (size 1.27 1.27)) hide)
     )
@@
       (effects (font (size 1.27 1.27)) (justify right))
     )
-    (property "Footprint" "Resistor_SMD:R_0603_1608Metric" (id 2) (at 185.42 73.66 0)
+    (property "Footprint" "Resistor_SMD:R_0402_1005Metric" (id 2) (at 185.42 73.66 0)
       (effects (font (size 1.27 1.27)) hide)
     )
@@
       (effects (font (size 1.27 1.27)) (justify right))
     )
-    (property "Footprint" "Resistor_SMD:R_0603_1608Metric" (id 2) (at 160.02 73.66 0)
+    (property "Footprint" "Resistor_SMD:R_0402_1005Metric" (id 2) (at 160.02 73.66 0)
       (effects (font (size 1.27 1.27)) hide)
     )
@@
       (effects (font (size 1.27 1.27)) (justify right))
     )
-    (property "Footprint" "Resistor_SMD:R_0603_1608Metric" (id 2) (at 172.72 57.15 0)
+    (property "Footprint" "Resistor_SMD:R_0402_1005Metric" (id 2) (at 172.72 57.15 0)
       (effects (font (size 1.27 1.27)) hide)
     )
@@
       (effects (font (size 1.27 1.27)) (justify right))
     )
-    (property "Footprint" "Resistor_SMD:R_0603_1608Metric" (id 2) (at 160.02 81.28 0)
+    (property "Footprint" "Resistor_SMD:R_0402_1005Metric" (id 2) (at 160.02 81.28 0)
       (effects (font (size 1.27 1.27)) hide)
     )
@@
       (effects (font (size 1.27 1.27)) (justify right))
     )
-    (property "Footprint" "Resistor_SMD:R_0603_1608Metric" (id 2) (at 121.92 49.53 0)
+    (property "Footprint" "Resistor_SMD:R_0402_1005Metric" (id 2) (at 121.92 49.53 0)
       (effects (font (size 1.27 1.27)) hide)
     )
@@
       (effects (font (size 1.27 1.27)) (justify right))
     )
-    (property "Footprint" "Resistor_SMD:R_0603_1608Metric" (id 2) (at 109.22 81.28 0)
+    (property "Footprint" "Resistor_SMD:R_0402_1005Metric" (id 2) (at 109.22 81.28 0)
       (effects (font (size 1.27 1.27)) hide)
     )
@@
       (effects (font (size 1.27 1.27)) (justify right))
     )
-    (property "Footprint" "Resistor_SMD:R_0603_1608Metric" (id 2) (at 109.22 73.66 0)
+    (property "Footprint" "Resistor_SMD:R_0402_1005Metric" (id 2) (at 109.22 73.66 0)
       (effects (font (size 1.27 1.27)) hide)
     )
@@
       (effects (font (size 1.27 1.27)) (justify right))
     )
-    (property "Footprint" "Resistor_SMD:R_0603_1608Metric" (id 2) (at 147.32 57.15 0)
+    (property "Footprint" "Resistor_SMD:R_0402_1005Metric" (id 2) (at 147.32 57.15 0)
       (effects (font (size 1.27 1.27)) hide)
     )
@@
       (effects (font (size 1.27 1.27)) (justify right))
     )
-    (property "Footprint" "Resistor_SMD:R_0603_1608Metric" (id 2) (at 147.32 49.53 0)
+    (property "Footprint" "Resistor_SMD:R_0402_1005Metric" (id 2) (at 147.32 49.53 0)
       (effects (font (size 1.27 1.27)) hide)
     )
@@
       (effects (font (size 1.27 1.27)) (justify right))
     )
-    (property "Footprint" "Resistor_SMD:R_0603_1608Metric" (id 2) (at 96.52 49.53 0)
-      (effects (font (size 1.27 1.27)) hide)
-    )
+    (property "Footprint" "Resistor_SMD:R_0402_1005Metric" (id 2) (at 96.52 49.53 0)
+      (effects (font (size 1.27 1.27)) hide)
+    )
