File: LightDrum/RGB_Control-3.kicad_sch (KiCad schematic)
At the start: 25 parts, among them Q501 PMXB43UNEZ, Q502 PMXB43UNEZ, Q503 PMXB43UNEZ, Q504 PMXB43UNEZ, Q505 PMXB43UNEZ, Q506 PMXB43UNEZ, Q507 PMXB43UNEZ, Q508 PMXB43UNEZ, U501 PCA9634_TSSOP20

Commit message: Replace relays and SWD conn
Other:
- note removed: "Screwed up the address transfer. Its currently the same as Strip Controller A 0x2A (42) Changed address to 0x2C (44)"
Changed lines of the file:
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@@
     (stroke (width 0) (type default))
-  )
-  (polyline (pts (xy 57.15 80.01) (xy 20.32 80.01))
-    (stroke (width 0) (type solid))
   )
   (polyline (pts (xy 16.51 16.51) (xy 16.51 92.71))
@@
     (stroke (width 0) (type default))
   )
-  (polyline (pts (xy 20.32 80.01) (xy 20.32 48.26))
-    (stroke (width 0) (type solid))
-  )
   (wire (pts (xy 34.29 35.56) (xy 36.83 35.56))
     (stroke (width 0) (type default))
@@
   (bus (pts (xy 165.1 64.77) (xy 182.88 64.77))
     (stroke (width 0) (type default))
-  )
-  (polyline (pts (xy 20.32 48.26) (xy 26.67 48.26))
-    (stroke (width 0) (type solid))
   )
   (wire (pts (xy 34.29 46.99) (xy 36.83 46.99))
@@
   (text "RGB STRIP CONTROLLER C" (at 16.51 20.32 0)
     (effects (font (size 2 2)) (justify left bottom))
-  )
-  (text "Screwed up the address transfer.\nIts currently the same as\nStrip Controller A 0x2A (42)\nChanged address to 0x2C (44)"
-    (at 20.828 79.502 0)
-    (effects (font (size 1.27 1.27)) (justify left bottom))
   )
   (label "LED8-G-SIG" (at 96.52 45.72 0) (fields_autoplaced)
@@
     (effects (font (size 1.27 1.27)) (justify left))
   )
+  (netclass_flag "" (length 2.54) (shape round) (at 71.12 64.77 180) (fields_autoplaced)
+    (effects (font (size 1.27 1.27)) (justify right bottom))
+    (property "Netclass" "LED-CTRL" (at 71.8185 67.31 0)
+      (effects (font (size 1.27 1.27) italic) (justify left))
+    )
+  )
   (symbol (lib_id "Device:R_Small_US") (at 134.62 73.66 0) (unit 1)

Commit message: Preliminary schematic lock - Starting PCB layout
Parts:
- Q501, Q502, Q503, Q504, Q505, Q506, Q507, Q508: SupplierPN (none) -> 1727-PMXB43UNEZCT-ND
- R501, R502, R503, R504, R509, R510, R511, R512: SupplierPN (none) -> RMCF0402FT100RCT-ND
- R505, R506, R507, R508, R513, R514, R515, R516: SupplierPN (none) -> 311-10KJRCT-ND
- U501: SupplierPN (none) -> 568-4066-1-ND
Connections:
- net I2C-SCLK renamed FI2C-SCLK_{S}
- net I2C-SDA renamed FI2C-SDA_{S}
- net ~{OE} renamed PWM-~{OE}_{PWM}
Changed lines of the file:
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@@
   (title_block
     (title "LightDrum")
-    (rev "REV10")
+    (rev "REV11")
     (company "Daxxn Industries")
   )
@@
     (effects (font (size 1.27 1.27)) (justify left bottom))
   )
-  (global_label "I2C-SCLK" (shape input) (at 34.29 33.02 180) (fields_autoplaced)
-    (effects (font (size 1.1 1.1) (thickness 0.254) bold) (justify right))
-    (property "Intersheetrefs" "${INTERSHEET_REFS}" (at 23.7956 32.893 0)
-      (effects (font (size 1.1 1.1) (thickness 0.254) bold) (justify right) hide)
-    )
-  )
-  (global_label "I2C-SDA" (shape input) (at 34.29 35.56 180) (fields_autoplaced)
-    (effects (font (size 1.1 1.1) (thickness 0.254) bold) (justify right))
-    (property "Intersheetrefs" "${INTERSHEET_REFS}" (at 24.8432 35.433 0)
-      (effects (font (size 1.1 1.1) (thickness 0.254) bold) (justify right) hide)
-    )
-  )
   (hierarchical_label "LED8-G" (shape output) (at 102.87 48.26 0) (fields_autoplaced)
     (effects (font (size 1.27 1.27)) (justify left))
   )
-  (hierarchical_label "~{OE}" (shape input) (at 34.29 38.1 180) (fields_autoplaced)
+  (hierarchical_label "PWM-~{OE}_{PWM}" (shape input) (at 34.29 38.1 180) (fields_autoplaced)
     (effects (font (size 1.27 1.27)) (justify right))
   )
@@
     (effects (font (size 1.27 1.27)) (justify left))
   )
+  (hierarchical_label "FI2C-SCLK_{S}" (shape input) (at 34.29 33.02 180) (fields_autoplaced)
+    (effects (font (size 1.27 1.27)) (justify right))
+  )
   (hierarchical_label "LED3-B" (shape output) (at 179.07 48.26 0) (fields_autoplaced)
     (effects (font (size 1.27 1.27)) (justify left))
@@
   (hierarchical_label "LED8-B" (shape output) (at 115.57 72.39 0) (fields_autoplaced)
     (effects (font (size 1.27 1.27)) (justify left))
+  )
+  (hierarchical_label "FI2C-SDA_{S}" (shape input) (at 34.29 35.56 180) (fields_autoplaced)
+    (effects (font (size 1.27 1.27)) (justify right))
   )
   (hierarchical_label "LED8-R" (shape output) (at 166.37 72.39 0) (fields_autoplaced)
@@
       (effects (font (size 1.27 1.27)) hide)
     )
+    (property "SupplierPN" "RMCF0402FT100RCT-ND" (at 134.62 73.66 0)
+      (effects (font (size 1.27 1.27)) hide)
+    )
     (pin "1")
     (pin "2")
@@
     (property "PartNumber" "0806-0003" (at 46.99 22.86 0)
       (effects (font (size 1.27 1.27)) (justify left))
+    )
+    (property "SupplierPN" "568-4066-1-ND" (at 45.72 44.45 0)
+      (effects (font (size 1.27 1.27)) hide)
     )
     (pin "1")
@@
       (effects (font (size 1.27 1.27)) (justify left))
     )
+    (property "SupplierPN" "1727-PMXB43UNEZCT-ND" (at 176.53 53.34 0)
+      (effects (font (size 1.27 1.27)) hide)
+    )
     (pin "1")
     (pin "2")
@@
       (effects (font (size 1.27 1.27)) hide)
     )
+    (property "SupplierPN" "RMCF0402FT100RCT-ND" (at 172.72 49.53 0)
+      (effects (font (size 1.27 1.27)) hide)
+    )
     (pin "1")
     (pin "2")
@@
       (effects (font (size 1.27 1.27)) (justify left))
     )
+    (property "SupplierPN" "1727-PMXB43UNEZCT-ND" (at 138.43 77.47 0)
+      (effects (font (size 1.27 1.27)) hide)
+    )
     (pin "1")
     (pin "2")
@@
       (effects (font (size 1.27 1.27)) hide)
     )
+    (property "SupplierPN" "311-10KJRCT-ND" (at 134.62 81.28 0)
+      (effects (font (size 1.27 1.27)) hide)
+    )
     (pin "1")
     (pin "2")
@@
       (effects (font (size 1.27 1.27)) hide)
     )
+    (property "SupplierPN" "311-10KJRCT-ND" (at 96.52 57.15 0)
+      (effects (font (size 1.27 1.27)) hide)
+    )
     (pin "1")
     (pin "2")
@@
       (effects (font (size 1.27 1.27)) (justify left))
     )
+    (property "SupplierPN" "1727-PMXB43UNEZCT-ND" (at 189.23 77.47 0)
+      (effects (font (size 1.27 1.27)) hide)
+    )
     (pin "1")
     (pin "2")
@@
       (effects (font (size 1.27 1.27)) (justify left))
     )
+    (property "SupplierPN" "1727-PMXB43UNEZCT-ND" (at 125.73 53.34 0)
+      (effects (font (size 1.27 1.27)) hide)
+    )
     (pin "1")
     (pin "2")
@@
       (effects (font (size 1.27 1.27)) hide)
     )
+    (property "SupplierPN" "311-10KJRCT-ND" (at 185.42 81.28 0)
+      (effects (font (size 1.27 1.27)) hide)
+    )
     (pin "1")
     (pin "2")
@@
       (effects (font (size 1.27 1.27)) hide)
     )
+    (property "SupplierPN" "311-10KJRCT-ND" (at 121.92 57.15 0)
+      (effects (font (size 1.27 1.27)) hide)
+    )
     (pin "1")
     (pin "2")
@@
     )
     (property "Datasheet" "~" (at 185.42 73.66 0)
+      (effects (font (size 1.27 1.27)) hide)
+    )
+    (property "SupplierPN" "RMCF0402FT100RCT-ND" (at 185.42 73.66 0)
       (effects (font (size 1.27 1.27)) hide)
     )
@@
       (effects (font (size 1.27 1.27)) hide)
     )
+    (property "SupplierPN" "RMCF0402FT100RCT-ND" (at 160.02 73.66 0)
+      (effects (font (size 1.27 1.27)) hide)
+    )
     (pin "1")
     (pin "2")
@@
       (effects (font (size 1.27 1.27)) (justify left))
     )
+    (property "SupplierPN" "1727-PMXB43UNEZCT-ND" (at 151.13 53.34 0)
+      (effects (font (size 1.27 1.27)) hide)
+    )
     (pin "1")
     (pin "2")
@@
     (property "PartNumber" "0703-0003" (at 115.57 73.66 0)
       (effects (font (size 1.27 1.27)) (justify left))
+    )
+    (property "SupplierPN" "1727-PMXB43UNEZCT-ND" (at 113.03 77.47 0)
+      (effects (font (size 1.27 1.27)) hide)
     )
     (pin "1")
@@
       (effects (font (size 1.27 1.27)) hide)
     )
+    (property "SupplierPN" "311-10KJRCT-ND" (at 172.72 57.15 0)
+      (effects (font (size 1.27 1.27)) hide)
+    )
     (pin "1")
     (pin "2")
@@
       (effects (font (size 1.27 1.27)) (justify left))
     )
+    (property "SupplierPN" "1727-PMXB43UNEZCT-ND" (at 100.33 53.34 0)
+      (effects (font (size 1.27 1.27)) hide)
+    )
     (pin "1")
     (pin "2")
@@
       (effects (font (size 1.27 1.27)) hide)
     )
+    (property "SupplierPN" "311-10KJRCT-ND" (at 160.02 81.28 0)
+      (effects (font (size 1.27 1.27)) hide)
+    )
     (pin "1")
     (pin "2")
@@
       (effects (font (size 1.27 1.27)) hide)
     )
+    (property "SupplierPN" "RMCF0402FT100RCT-ND" (at 121.92 49.53 0)
+      (effects (font (size 1.27 1.27)) hide)
+    )
     (pin "1")
     (pin "2")
@@
     )
     (property "Datasheet" "~" (at 109.22 81.28 0)
+      (effects (font (size 1.27 1.27)) hide)
+    )
+    (property "SupplierPN" "311-10KJRCT-ND" (at 109.22 81.28 0)
       (effects (font (size 1.27 1.27)) hide)
     )
@@
       (effects (font (size 1.27 1.27)) (justify left))
     )
+    (property "SupplierPN" "1727-PMXB43UNEZCT-ND" (at 163.83 77.47 0)
+      (effects (font (size 1.27 1.27)) hide)
+    )
     (pin "1")
     (pin "2")
@@
       (effects (font (size 1.27 1.27)) hide)
     )
+    (property "SupplierPN" "RMCF0402FT100RCT-ND" (at 109.22 73.66 0)
+      (effects (font (size 1.27 1.27)) hide)
+    )
     (pin "1")
     (pin "2")
@@
       (effects (font (size 1.27 1.27)) hide)
     )
+    (property "SupplierPN" "311-10KJRCT-ND" (at 147.32 57.15 0)
+      (effects (font (size 1.27 1.27)) hide)
+    )
     (pin "1")
     (pin "2")
@@
       (effects (font (size 1.27 1.27)) hide)
     )
+    (property "SupplierPN" "RMCF0402FT100RCT-ND" (at 147.32 49.53 0)
+      (effects (font (size 1.27 1.27)) hide)
+    )
     (pin "1")
     (pin "2")
@@
       (effects (font (size 1.27 1.27)) hide)
     )
+    (property "SupplierPN" "RMCF0402FT100RCT-ND" (at 96.52 49.53 0)
+      (effects (font (size 1.27 1.27)) hide)
+    )

Commit message: Component placement complete
Parts:
- renumbered Q501 to Q20, Q502 to Q21, Q503 to Q22, Q504 to Q23, Q505 to Q24, Q506 to Q25, Q507 to Q26, Q508 to Q27, R501 to R84, R502 to R85, R503 to R86, R504 to R87, R505 to R88, R506 to R89, R507 to R90, R508 to R91, R509 to R92, R510 to R93, R511 to R94, R512 to R95, R513 to R96, R514 to R97, R515 to R98, R516 to R99, U501 to U11

Commit message: First draft layout almost complete
Connections:
- net LED4-B-SIG: now also U11.7 (LED1); no longer U11.8 (LED2)
- net LED4-R-SIG: now also U11.9 (LED3); no longer U11.6 (LED0)
- net LED8-B-SIG: now also U11.6 (LED0); no longer U11.9 (LED3)
- net LED8-R-SIG: now also U11.8 (LED2); no longer U11.7 (LED1)
Changed lines of the file:
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@@
     (effects (font (size 1.27 1.27)) (justify left bottom))
   )
-  (label "LED4-B-SIG" (at 55.88 40.64 0) (fields_autoplaced)
+  (label "LED4-B-SIG" (at 55.88 38.1 0) (fields_autoplaced)
     (effects (font (size 1.27 1.27)) (justify left bottom))
   )
@@
     (effects (font (size 1.27 1.27)) (justify left bottom))
   )
-  (label "LED8-B-SIG" (at 55.88 43.18 0) (fields_autoplaced)
+  (label "LED8-B-SIG" (at 55.88 35.56 0) (fields_autoplaced)
     (effects (font (size 1.27 1.27)) (justify left bottom))
   )
@@
     (effects (font (size 1.27 1.27)) (justify left bottom))
   )
-  (label "LED4-R-SIG" (at 55.88 35.56 0) (fields_autoplaced)
+  (label "LED4-R-SIG" (at 55.88 43.18 0) (fields_autoplaced)
     (effects (font (size 1.27 1.27)) (justify left bottom))
   )
-  (label "LED8-R-SIG" (at 55.88 38.1 0) (fields_autoplaced)
+  (label "LED8-R-SIG" (at 55.88 40.64 0) (fields_autoplaced)
     (effects (font (size 1.27 1.27)) (justify left bottom))
   )

Commit message: Minor fixes and cleanup - REV11
Parts:
- added C75, C76: 100nF, Capacitor_SMD:C_0402_1005Metric, symbol Daxxn_Device:C
Connections:
- net GND: now also C75.2, C76.2
- net VDD: now also C75.1, C76.1
Other:
- moved on the sheet: Q20, Q21, Q22, Q23, Q24, Q25, Q26, Q27, R84, R85, R86, R87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

Commit message: Replace DSub with much better ECU conn
Parts:
- removed C75, C76: 100nF, Capacitor_SMD:C_0402_1005Metric, symbol Daxxn_Device:C
- removed Q20, Q21, Q22, Q23, Q24, Q25, Q26, Q27: PMXB43UNEZ, Daxxn_Packages:DFN1010D-3, symbol Daxxn_Transistors:PMXB43UNEZ
- removed R84, R85, R86, R87, R92, R93, R94, R95: 100, Resistor_SMD:R_0402_1005Metric, symbol Device:R_Small_US
- removed R88, R89, R90, R91, R96, R97, R98, R99: 10K, Resistor_SMD:R_0402_1005Metric, symbol Device:R_Small_US
- removed U11: PCA9634_TSSOP20, Package_SO:TSSOP-20_4.4x6.5mm_P0.65mm, symbol Daxxn_IC:PCA9634_TSSOP20
Other:
- note removed: "Address: 44 0x2C"
- note removed: "RGB STRIP CONTROLLER C"
