File: LightDrum/RGB_Control.kicad_sch (KiCad schematic)
At the start: 0 parts

Commit message: Add docs and gerbers for REV7
Other:
- title: RGB STRIP CONNECTOR -> LightDrum
Changed lines of the file:
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@@
   (paper "A4")
   (title_block
-    (title "RGB STRIP CONNECTOR")
-    (rev "REV6")
+    (title "LightDrum")
+    (rev "REV7")
     (company "Daxxn Industries")
   )

Commit message: First pass over schematic (WIP)
Other:
- removed sheet Strip MUX
Changed lines of the file:
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@@
   (title_block
     (title "LightDrum")
-    (rev "REV7")
+    (rev "REV8")
     (company "Daxxn Industries")
   )
+  (junction (at 46.99 119.38) (diameter 0) (color 0 0 0 0)
+  )
+  (junction (at 27.94 119.38) (diameter 0) (color 0 0 0 0)
+  )
   (wire (pts (xy 85.09 67.31) (xy 97.79 67.31))
     (stroke (width 0) (type default) (color 0 0 0 0))
@@
     (stroke (width 0) (type default) (color 0 0 0 0))
   )
-  (wire (pts (xy 72.39 116.84) (xy 72.39 129.54))
-    (stroke (width 0) (type default) (color 0 0 0 0))
-  )
   (wire (pts (xy 59.69 46.99) (xy 97.79 46.99))
     (stroke (width 0) (type default) (color 0 0 0 0))
@@
     (stroke (width 0) (type solid) (color 0 0 0 0))
   )
+  (wire (pts (xy 21.59 110.49) (xy 27.94 110.49))
+    (stroke (width 0) (type default) (color 0 0 0 0))
+  )
   (polyline (pts (xy 218.44 128.27) (xy 218.44 132.08))
     (stroke (width 0) (type solid) (color 0 0 0 0))
@@
     (stroke (width 0) (type solid) (color 0 0 0 0))
   )
+  (wire (pts (xy 46.99 102.87) (xy 46.99 119.38))
+    (stroke (width 0) (type default) (color 0 0 0 0))
+  )
   (wire (pts (xy 156.21 35.56) (xy 157.48 35.56))
     (stroke (width 0) (type default) (color 0 0 0 0))
   )
-  (wire (pts (xy 21.59 134.62) (xy 21.59 88.9))
+  (wire (pts (xy 21.59 88.9) (xy 21.59 110.49))
+    (stroke (width 0) (type default) (color 0 0 0 0))
+  )
+  (wire (pts (xy 27.94 110.49) (xy 27.94 119.38))
     (stroke (width 0) (type default) (color 0 0 0 0))
   )
@@
     (stroke (width 0) (type default) (color 0 0 0 0))
   )
+  (wire (pts (xy 72.39 116.84) (xy 72.39 119.38))
+    (stroke (width 0) (type default) (color 0 0 0 0))
+  )
   (wire (pts (xy 34.29 35.56) (xy 97.79 35.56))
     (stroke (width 0) (type default) (color 0 0 0 0))
@@
     (stroke (width 0) (type default) (color 0 0 0 0))
   )
-  (wire (pts (xy 74.93 129.54) (xy 72.39 129.54))
-    (stroke (width 0) (type default) (color 0 0 0 0))
-  )
   (wire (pts (xy 85.09 58.42) (xy 97.79 58.42))
     (stroke (width 0) (type default) (color 0 0 0 0))
@@
     (stroke (width 0) (type default) (color 0 0 0 0))
   )
-  (wire (pts (xy 46.99 132.08) (xy 46.99 102.87))
-    (stroke (width 0) (type default) (color 0 0 0 0))
-  )
   (polyline (pts (xy 118.11 16.51) (xy 175.26 16.51))
     (stroke (width 0) (type default) (color 0 0 0 0))
@@
     (stroke (width 0) (type default) (color 0 0 0 0))
   )
+  (wire (pts (xy 26.67 119.38) (xy 27.94 119.38))
+    (stroke (width 0) (type default) (color 0 0 0 0))
+  )
   (polyline (pts (xy 120.65 139.7) (xy 129.54 139.7))
     (stroke (width 0) (type solid) (color 0 0 0 0))
@@
     (stroke (width 0) (type default) (color 0 0 0 0))
   )
+  (wire (pts (xy 46.99 119.38) (xy 72.39 119.38))
+    (stroke (width 0) (type default) (color 0 0 0 0))
+  )
   (wire (pts (xy 34.29 76.2) (xy 97.79 76.2))
     (stroke (width 0) (type default) (color 0 0 0 0))
   )
-  (wire (pts (xy 72.39 140.97) (xy 74.93 140.97))
-    (stroke (width 0) (type default) (color 0 0 0 0))
-  )
   (polyline (pts (xy 118.11 16.51) (xy 118.11 121.92))
     (stroke (width 0) (type default) (color 0 0 0 0))
@@
     (stroke (width 0) (type solid) (color 0 0 0 0))
   )
-  (wire (pts (xy 74.93 134.62) (xy 21.59 134.62))
-    (stroke (width 0) (type default) (color 0 0 0 0))
-  )
   (polyline (pts (xy 175.26 16.51) (xy 175.26 121.92))
     (stroke (width 0) (type default) (color 0 0 0 0))
@@
     (stroke (width 0) (type solid) (color 0 0 0 0))
   )
+  (wire (pts (xy 27.94 119.38) (xy 46.99 119.38))
+    (stroke (width 0) (type default) (color 0 0 0 0))
+  )
   (polyline (pts (xy 118.11 121.92) (xy 91.44 121.92))
     (stroke (width 0) (type default) (color 0 0 0 0))
@@
     (stroke (width 0) (type solid) (color 0 0 0 0))
   )
-  (wire (pts (xy 74.93 132.08) (xy 46.99 132.08))
-    (stroke (width 0) (type default) (color 0 0 0 0))
-  )
   (polyline (pts (xy 91.44 121.92) (xy 16.51 121.92))
-    (stroke (width 0) (type default) (color 0 0 0 0))
-  )
-  (wire (pts (xy 72.39 138.43) (xy 74.93 138.43))
     (stroke (width 0) (type default) (color 0 0 0 0))
   )
@@
     (effects (font (size 2.5 2.5) bold) (justify left bottom))
   )
-  (hierarchical_label "MUX-BYPASS" (shape input) (at 72.39 138.43 180)
+  (hierarchical_label "STRIP5-CURR" (shape output) (at 157.48 38.1 0)
+    (effects (font (size 1.27 1.27)) (justify left))
+  )
+  (hierarchical_label "~{PWM-OE}" (shape input) (at 26.67 119.38 180)
     (effects (font (size 1.27 1.27)) (justify right))
   )
-  (hierarchical_label "STRIP5-CURR" (shape output) (at 157.48 38.1 0)
-    (effects (font (size 1.27 1.27)) (justify left))
-  )
   (hierarchical_label "STRIP7-CURR" (shape output) (at 157.48 43.18 0)
     (effects (font (size 1.27 1.27)) (justify left))
@@
   (hierarchical_label "STRIP3-CURR" (shape output) (at 157.48 33.02 0)
     (effects (font (size 1.27 1.27)) (justify left))
-  )
-  (hierarchical_label "MUX-ENABLE" (shape input) (at 72.39 140.97 180)
-    (effects (font (size 1.27 1.27)) (justify right))
   )
   (hierarchical_label "STRIP2-CURR" (shape output) (at 157.48 30.48 0)
@@
       (effects (font (size 1.27 1.27)) (justify left))
     )
-  )
-  (sheet (at 74.93 127) (size 20.32 16.51)
-    (stroke (width 0.1524) (type solid) (color 0 0 0 0))
-    (fill (color 0 0 0 0.0000))
-    (property "Sheet name" "Strip MUX" (id 0) (at 74.93 127 0)
-      (effects (font (size 1.27 1.27)) (justify left bottom))
-    )
-    (property "Sheet file" "LED_MUX.kicad_sch" (id 1) (at 74.93 144.78 0)
-      (effects (font (size 0.5 0.5)) (justify left top))
-    )
-    (pin "PWM-OE-1" output (at 74.93 134.62 180)
-      (effects (font (size 1.27 1.27)) (justify left))
-    )
-    (pin "PWM-OE-2" output (at 74.93 132.08 180)
-      (effects (font (size 1.27 1.27)) (justify left))
-    )
-    (pin "PWM-OE-3" output (at 74.93 129.54 180)
-      (effects (font (size 1.27 1.27)) (justify left))
-    )
-    (pin "BYPASS" input (at 74.93 138.43 180)
-      (effects (font (size 1.27 1.27)) (justify left))
-    )
-    (pin "ENABLE" input (at 74.93 140.97 180)
-      (effects (font (size 1.27 1.27)) (justify left))
-    )

Commit message: Clean up and remove old files
Other:
- sheet Strip Connector: file LED_Connector.kicad_sch -> Strip_Connector.kicad_sch
Changed lines of the file:
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@@
       (effects (font (size 1.27 1.27)) (justify left bottom))
     )
-    (property "Sheet file" "LED_Connector.kicad_sch" (id 1) (at 97.79 118.3866 0)
+    (property "Sheet file" "Strip_Connector.kicad_sch" (id 1) (at 97.79 118.3866 0)
       (effects (font (size 0.5 0.5)) (justify left top))
     )

Commit message: interface layout completed - REV6
Other:
- sheet Strip Connector ports: added DMX+, DMX-; removed none
Changed lines of the file:
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@@
   (junction (at 46.99 119.38) (diameter 0) (color 0 0 0 0)
   )
-  (junction (at 27.94 119.38) (diameter 0) (color 0 0 0 0)
+  (junction (at 30.48 119.38) (diameter 0) (color 0 0 0 0)
   )
   (wire (pts (xy 85.09 67.31) (xy 97.79 67.31))
@@
     (stroke (width 0) (type solid) (color 0 0 0 0))
   )
-  (wire (pts (xy 21.59 110.49) (xy 27.94 110.49))
+  (wire (pts (xy 21.59 110.49) (xy 30.48 110.49))
     (stroke (width 0) (type default) (color 0 0 0 0))
   )
@@
     (stroke (width 0) (type default) (color 0 0 0 0))
   )
-  (wire (pts (xy 27.94 110.49) (xy 27.94 119.38))
+  (wire (pts (xy 30.48 110.49) (xy 30.48 119.38))
     (stroke (width 0) (type default) (color 0 0 0 0))
   )
@@
     (stroke (width 0) (type default) (color 0 0 0 0))
   )
-  (wire (pts (xy 26.67 119.38) (xy 27.94 119.38))
+  (wire (pts (xy 30.48 119.38) (xy 46.99 119.38))
     (stroke (width 0) (type default) (color 0 0 0 0))
   )
@@
     (stroke (width 0) (type solid) (color 0 0 0 0))
   )
-  (wire (pts (xy 27.94 119.38) (xy 46.99 119.38))
+  (wire (pts (xy 27.94 119.38) (xy 30.48 119.38))
     (stroke (width 0) (type default) (color 0 0 0 0))
   )
@@
     (stroke (width 0) (type solid) (color 0 0 0 0))
   )
+  (wire (pts (xy 96.52 125.73) (xy 97.79 125.73))
+    (stroke (width 0) (type default) (color 0 0 0 0))
+  )
   (polyline (pts (xy 91.44 121.92) (xy 16.51 121.92))
+    (stroke (width 0) (type default) (color 0 0 0 0))
+  )
+  (wire (pts (xy 96.52 128.27) (xy 97.79 128.27))
     (stroke (width 0) (type default) (color 0 0 0 0))
   )
@@
     (effects (font (size 1.27 1.27)) (justify left))
   )
-  (hierarchical_label "~{PWM-OE}" (shape input) (at 26.67 119.38 180)
+  (hierarchical_label "~{PWM-OE}" (shape input) (at 27.94 119.38 180)
     (effects (font (size 1.27 1.27)) (justify right))
   )
@@
     (effects (font (size 1.27 1.27)) (justify left))
   )
+  (hierarchical_label "DMX+" (shape bidirectional) (at 96.52 128.27 180)
+    (effects (font (size 1.27 1.27)) (justify right))
+  )
   (hierarchical_label "STRIP3-CURR" (shape output) (at 157.48 33.02 0)
     (effects (font (size 1.27 1.27)) (justify left))
@@
   (hierarchical_label "STRIP4-CURR" (shape output) (at 157.48 35.56 0)
     (effects (font (size 1.27 1.27)) (justify left))
+  )
+  (hierarchical_label "DMX-" (shape bidirectional) (at 96.52 125.73 180)
+    (effects (font (size 1.27 1.27)) (justify right))
   )
   (sheet (at 69.85 57.15) (size 15.24 59.69)
@@
     )
   )
-  (sheet (at 97.79 25.4) (size 13.97 92.71) (fields_autoplaced)
+  (sheet (at 97.79 25.4) (size 13.97 105.41) (fields_autoplaced)
     (stroke (width 0.1524) (type solid) (color 0 0 0 0))
     (fill (color 0 0 0 0.0000))
@@
       (effects (font (size 1.27 1.27)) (justify left bottom))
     )
-    (property "Sheet file" "Strip_Connector.kicad_sch" (id 1) (at 97.79 118.3866 0)
+    (property "Sheet file" "Strip_Connector.kicad_sch" (id 1) (at 97.79 131.0866 0)
       (effects (font (size 0.5 0.5)) (justify left top))
     )
@@
       (effects (font (size 1.27 1.27)) (justify left))
     )
+    (pin "DMX-" bidirectional (at 97.79 125.73 180)
+      (effects (font (size 1.27 1.27)) (justify left))
+    )
+    (pin "DMX+" bidirectional (at 97.79 128.27 180)
+      (effects (font (size 1.27 1.27)) (justify left))
+    )
