File: LightDrum/TestPoints.kicad_sch (KiCad schematic)
At the start: 6 parts

Commit message: interface layout completed - REV6
Parts:
- added TP1201: XLR REF TP, Connector_PinHeader_2.54mm:PinHeader_1x02_P2.54mm_Vertical, symbol Connector:TestPoint_2Pole
- added TP1202: HP REF TP, Connector_PinHeader_2.54mm:PinHeader_1x02_P2.54mm_Vertical, symbol Connector:TestPoint_2Pole
- added TPA1201: VDRIVE TP, TestPoint:TestPoint_Loop_D2.54mm_Drill1.5mm_Beaded, symbol Connector:TestPoint_Alt
Connections:
- net GND: now also TP1201.2, TP1202.2
- new net HP-REF: TP1202.1
- new net Vdrive: TPA1201.1
- new net XLR-REF: TP1201.1
Other:
- note added: "POWER"
- note added: "SIGNALS"
- moved on the sheet: TP1101, TP1102, TPA1101, TPA1102, TPA1103, TPA1104

Commit message: Add main page to sch and xlr audio input diff-amp
Parts:
- removed TP1201: XLR REF TP, Connector_PinHeader_2.54mm:PinHeader_1x02_P2.54mm_Vertical, symbol Connector:TestPoint_2Pole
- removed TP1202: HP REF TP, Connector_PinHeader_2.54mm:PinHeader_1x02_P2.54mm_Vertical, symbol Connector:TestPoint_2Pole
- added TPA1301: XLR TP, TestPoint:TestPoint_Pad_D1.5mm, symbol Connector:TestPoint_Alt
- added TPA1302: HP TP, TestPoint:TestPoint_Pad_D1.5mm, symbol Connector:TestPoint_Alt
Connections:
- net HP-REF: now also TPA1302.1
- net XLR-REF: now also TPA1301.1
Changed lines of the file:
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@@
-    (stroke (width 0) (type default) (color 0 0 0 0))
-  )
-  (wire (pts (xy 38.1 40.64) (xy 40.64 40.64))
-    (stroke (width 0) (type default) (color 0 0 0 0))
-  )
-  (wire (pts (xy 40.64 49.53) (xy 40.64 50.8))
     (stroke (width 0) (type default) (color 0 0 0 0))
   )
@@
     (stroke (width 0) (type default) (color 0 0 0 0))
   )
-  (wire (pts (xy 40.64 40.64) (xy 40.64 41.91))
-    (stroke (width 0) (type default) (color 0 0 0 0))
-  )
   (polyline (pts (xy 52.07 16.51) (xy 52.07 62.23))
     (stroke (width 0) (type default) (color 0 0 0 0))
@@
   )
   (wire (pts (xy 25.4 49.53) (xy 27.94 49.53))
-    (stroke (width 0) (type default) (color 0 0 0 0))
-  )
-  (wire (pts (xy 38.1 49.53) (xy 40.64 49.53))
     (stroke (width 0) (type default) (color 0 0 0 0))
   )
@@
     (effects (font (size 1.27 1.27)) (justify right))
   )
-  (symbol (lib_id "power:GND") (at 40.64 41.91 0) (unit 1)
-    (in_bom yes) (on_board yes)
-    (property "Reference" "#PWR0145" (id 0) (at 40.64 48.26 0)
-      (effects (font (size 1.27 1.27)) hide)
-    )
-    (property "Value" "GND" (id 1) (at 40.64 45.72 0))
-    (property "Footprint" "" (id 2) (at 40.64 41.91 0)
-      (effects (font (size 1.27 1.27)) hide)
-    )
-    (property "Datasheet" "" (id 3) (at 40.64 41.91 0)
-      (effects (font (size 1.27 1.27)) hide)
-    )
-    (pin "1")
-  )
   (symbol (lib_id "Connector:TestPoint_2Pole") (at 33.02 25.4 0) (unit 1)
     (in_bom yes) (on_board yes)
@@
     (pin "1")
   )
-  (symbol (lib_id "power:GND") (at 40.64 50.8 0) (unit 1)
-    (in_bom yes) (on_board yes)
-    (property "Reference" "#PWR0146" (id 0) (at 40.64 57.15 0)
-      (effects (font (size 1.27 1.27)) hide)
-    )
-    (property "Value" "GND" (id 1) (at 40.64 54.61 0))
-    (property "Footprint" "" (id 2) (at 40.64 50.8 0)
-      (effects (font (size 1.27 1.27)) hide)
-    )
-    (property "Datasheet" "" (id 3) (at 40.64 50.8 0)
-      (effects (font (size 1.27 1.27)) hide)
-    )
-    (pin "1")
-  )
-  (symbol (lib_id "Connector:TestPoint_2Pole") (at 33.02 49.53 0) (unit 1)
-    (in_bom yes) (on_board yes)
-    (property "Reference" "TP1202" (id 0) (at 33.02 48.006 0))
-    (property "Value" "HP REF TP" (id 1) (at 33.02 51.308 0))
-    (property "Footprint" "Connector_PinHeader_2.54mm:PinHeader_1x02_P2.54mm_Vertical" (id 2) (at 33.02 49.53 0)
-      (effects (font (size 1.27 1.27)) hide)
-    )
-    (property "Datasheet" "~" (id 3) (at 33.02 49.53 0)
-      (effects (font (size 1.27 1.27)) hide)
-    )
-    (pin "1")
-    (pin "2")
+  (symbol (lib_id "Connector:TestPoint_Alt") (at 27.94 49.53 270) (unit 1)
+    (in_bom yes) (on_board yes)
+    (property "Reference" "TPA1302" (id 0) (at 32.512 47.752 90)
+      (effects (font (size 1.27 1.27)) (justify left))
+    )
+    (property "Value" "HP TP" (id 1) (at 32.512 49.53 90)
+      (effects (font (size 1.27 1.27)) (justify left))
+    )
+    (property "Footprint" "TestPoint:TestPoint_Pad_D1.5mm" (id 2) (at 27.94 54.61 0)
+      (effects (font (size 1.27 1.27)) hide)
+    )
+    (property "Datasheet" "~" (id 3) (at 27.94 54.61 0)
+      (effects (font (size 1.27 1.27)) hide)
+    )
+    (pin "1")
   )
   (symbol (lib_id "Connector:TestPoint_Alt") (at 58.42 40.64 270) (unit 1)
@@
     )
     (property "Datasheet" "~" (id 3) (at 58.42 45.72 0)
+      (effects (font (size 1.27 1.27)) hide)
+    )
+    (pin "1")
+  )
+  (symbol (lib_id "Connector:TestPoint_Alt") (at 27.94 40.64 270) (unit 1)
+    (in_bom yes) (on_board yes)
+    (property "Reference" "TPA1301" (id 0) (at 32.512 38.862 90)
+      (effects (font (size 1.27 1.27)) (justify left))
+    )
+    (property "Value" "XLR TP" (id 1) (at 32.512 40.64 90)
+      (effects (font (size 1.27 1.27)) (justify left))
+    )
+    (property "Footprint" "TestPoint:TestPoint_Pad_D1.5mm" (id 2) (at 27.94 45.72 0)
+      (effects (font (size 1.27 1.27)) hide)
+    )
+    (property "Datasheet" "~" (id 3) (at 27.94 45.72 0)
       (effects (font (size 1.27 1.27)) hide)
     )
@@
     (pin "1")
   )
-  (symbol (lib_id "Connector:TestPoint_2Pole") (at 33.02 40.64 0) (unit 1)
-    (in_bom yes) (on_board yes)
-    (property "Reference" "TP1201" (id 0) (at 33.02 39.116 0))
-    (property "Value" "XLR REF TP" (id 1) (at 33.02 42.418 0))
-    (property "Footprint" "Connector_PinHeader_2.54mm:PinHeader_1x02_P2.54mm_Vertical" (id 2) (at 33.02 40.64 0)
-      (effects (font (size 1.27 1.27)) hide)
-    )
-    (property "Datasheet" "~" (id 3) (at 33.02 40.64 0)
-      (effects (font (size 1.27 1.27)) hide)
-    )
-    (pin "1")
-    (pin "2")
-  )
   (symbol (lib_id "Connector:TestPoint_Alt") (at 58.42 33.02 270) (unit 1)
