File: LightDrum/LED_Power_Control.kicad_sch (KiCad schematic)
At the start: 8 parts, among them J901 DIN-4-SH, K901 ALQ112, K902 ALQ112, U902 SSM3K361R_SOT23F

Commit message: Main and Interface PCBs locked - REV9
Parts:
- F901: value 10A -> 15A
Other:
- note added: "Uses new 12V 196W power supply. Both relays are required for incresing current capacity."
- note removed: "Due to the large current for the RGB strips, the load needs to be divided up between 2 barrel jacks. If only one is plugged in, it would probably melt. To prevent any melty firey and expensy issues, the RGB strips will not be powered unless both jacks are used AND the controller agrees."
- moved on the sheet: D901, F901, J901, K901, K902, R903, R904, U902

Commit message: Start REV 10 - Fix small issues
Parts:
- added R1008: 10K, Resistor_SMD:R_1206_3216Metric, symbol Device:R_Small_US
Connections:
- net GND: now also R1008.2
- net at F901.1, J901.1, J901.2: now also R1008.1
Changed lines of the file:
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@@
   (junction (at 60.96 36.83) (diameter 0) (color 0 0 0 0)
   )
+  (junction (at 40.64 43.18) (diameter 0) (color 0 0 0 0)
+  )
   (junction (at 81.28 36.83) (diameter 0) (color 0 0 0 0)
   )
@@
   )
   (junction (at 101.6 36.83) (diameter 0) (color 0 0 0 0)
+  )
+  (junction (at 40.64 48.26) (diameter 0) (color 0 0 0 0)
   )
   (junction (at 71.12 36.83) (diameter 0) (color 0 0 0 0)
@@
     (stroke (width 0) (type default) (color 0 0 0 0))
   )
+  (wire (pts (xy 40.64 43.18) (xy 45.72 43.18))
+    (stroke (width 0) (type default) (color 0 0 0 0))
+  )
+  (wire (pts (xy 40.64 48.26) (xy 45.72 48.26))
+    (stroke (width 0) (type default) (color 0 0 0 0))
+  )
   (wire (pts (xy 111.76 36.83) (xy 101.6 36.83))
     (stroke (width 0) (type default) (color 0 0 0 0))
@@
     (effects (font (size 1.27 1.27)) (justify right))
   )
+  (symbol (lib_id "Device:R_Small_US") (at 45.72 45.72 0) (unit 1)
+    (in_bom yes) (on_board yes)
+    (property "Reference" "R1008" (id 0) (at 44.45 44.958 0)
+      (effects (font (size 1.27 1.27)) (justify right))
+    )
+    (property "Value" "10K" (id 1) (at 44.45 46.736 0)
+      (effects (font (size 1.27 1.27)) (justify right))
+    )
+    (property "Footprint" "Resistor_SMD:R_1206_3216Metric" (id 2) (at 45.72 45.72 0)
+      (effects (font (size 1.27 1.27)) hide)
+    )
+    (property "Datasheet" "~" (id 3) (at 45.72 45.72 0)
+      (effects (font (size 1.27 1.27)) hide)
+    )
+    (pin "1")
+    (pin "2")
+  )
   (symbol (lib_id "Daxxn_Connectors:DIN-4-SH") (at 33.02 45.72 270) (unit 1)
