File: LightDrum/LightDrum.kicad_sch (KiCad schematic)
At the start: 5 parts, among them U1 STR485

Commit message: First draft layout almost complete
Connections:
- net DMX-EN is gone; now on net DMX-EN_{S}: U1.3 (DE), U1.4 (~{RE})
- net DMX-RX is gone; now on net DMX-RX_{S}: U1.2 (R)
- net DMX-TX is gone; now on net DMX-TX_{S}: U1.5 (D)
Other:
- sheet INTERFACE CONNECTOR ports: added MENU-ACT_{INT}, MENU-BACK_{INT}, MENU-DOWN_{INT}, MENU-LEFT_{INT}, MENU-RIGHT_{INT}, MENU-UP_{INT}; removed MENU-ACT, MENU-BACK, MENU-DOWN, MENU-LEFT, MENU-RIGHT, MENU-UP
Changed lines of the file:
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@@
     (effects (font (size 1.27 1.27)) (justify left bottom))
-  )
-  (label "MENU-ACT" (at 182.88 123.19 180) (fields_autoplaced)
-    (effects (font (size 1.27 1.27)) (justify right bottom))
   )
   (label "AUDIO-SRC-IND_{PWM}" (at 182.88 146.05 180) (fields_autoplaced)
@@
     (effects (font (size 1.27 1.27)) (justify left bottom))
   )
-  (label "MENU-UP" (at 182.88 115.57 180) (fields_autoplaced)
+  (label "DMX-TX_{S}" (at 24.13 144.78 0) (fields_autoplaced)
+    (effects (font (size 1.27 1.27)) (justify left bottom))
+  )
+  (label "MENU-UP_{INT}" (at 182.88 115.57 180) (fields_autoplaced)
     (effects (font (size 1.27 1.27)) (justify right bottom))
   )
@@
     (effects (font (size 1.27 1.27)) (justify left bottom))
   )
+  (label "ENC1-A_{INT}" (at 107.95 113.03 0) (fields_autoplaced)
+    (effects (font (size 1.27 1.27)) (justify left bottom))
+  )
   (label "ENC2-B" (at 15.24 69.85 0) (fields_autoplaced)
     (effects (font (size 1.27 1.27)) (justify left bottom))
@@
     (effects (font (size 1.27 1.27)) (justify right bottom))
   )
-  (label "ENC1-A" (at 107.95 113.03 0) (fields_autoplaced)
-    (effects (font (size 1.27 1.27)) (justify left bottom))
-  )
-  (label "ENC1-SW" (at 107.95 118.11 0) (fields_autoplaced)
-    (effects (font (size 1.27 1.27)) (justify left bottom))
-  )
-  (label "MENU-DOWN" (at 182.88 120.65 180) (fields_autoplaced)
-    (effects (font (size 1.27 1.27)) (justify right bottom))
-  )
   (label "I2C-SCLK_{S}" (at 107.95 144.78 0) (fields_autoplaced)
     (effects (font (size 1.27 1.27)) (justify left bottom))
@@
     (effects (font (size 1.27 1.27)) (justify left bottom))
   )
-  (label "ENC2-SW" (at 107.95 125.73 0) (fields_autoplaced)
-    (effects (font (size 1.27 1.27)) (justify left bottom))
-  )
   (label "SD-CD_{S}" (at 106.68 49.53 180) (fields_autoplaced)
     (effects (font (size 1.27 1.27)) (justify right bottom))
@@
     (effects (font (size 1.27 1.27)) (justify left bottom))
   )
+  (label "DMX-RX_{S}" (at 24.13 135.89 0) (fields_autoplaced)
+    (effects (font (size 1.27 1.27)) (justify left bottom))
+  )
   (label "GRAPH-LE_{S}" (at 182.88 134.62 180) (fields_autoplaced)
     (effects (font (size 1.27 1.27)) (justify right bottom))
@@
     (effects (font (size 1.27 1.27)) (justify left bottom))
   )
+  (label "MENU-LEFT_{INT}" (at 182.88 118.11 180) (fields_autoplaced)
+    (effects (font (size 1.27 1.27)) (justify right bottom))
+  )
   (label "MENU-UP_{INT}" (at 15.24 45.72 0) (fields_autoplaced)
     (effects (font (size 1.27 1.27)) (justify left bottom))
@@
     (effects (font (size 1.27 1.27)) (justify right bottom))
   )
+  (label "MENU-RIGHT_{INT}" (at 182.88 125.73 180) (fields_autoplaced)
+    (effects (font (size 1.27 1.27)) (justify right bottom))
+  )
   (label "I2C-SDA_{S}" (at 106.68 81.28 180) (fields_autoplaced)
     (effects (font (size 1.27 1.27)) (justify right bottom))
@@
     (effects (font (size 1.27 1.27)) (justify right bottom))
   )
+  (label "ENC1-SW_{INT}" (at 107.95 118.11 0) (fields_autoplaced)
+    (effects (font (size 1.27 1.27)) (justify left bottom))
+  )
+  (label "MENU-DOWN_{INT}" (at 182.88 120.65 180) (fields_autoplaced)
+    (effects (font (size 1.27 1.27)) (justify right bottom))
+  )
+  (label "MENU-BACK_{INT}" (at 182.88 113.03 180) (fields_autoplaced)
+    (effects (font (size 1.27 1.27)) (justify right bottom))
+  )
   (label "MENU-BACK_{INT}" (at 15.24 43.18 0) (fields_autoplaced)
     (effects (font (size 1.27 1.27)) (justify left bottom))
@@
     (effects (font (size 1.27 1.27)) (justify left bottom))
   )
+  (label "ENC2-SW_{INT}" (at 107.95 125.73 0) (fields_autoplaced)
+    (effects (font (size 1.27 1.27)) (justify left bottom))
+  )
   (label "SD-CLK_{S}" (at 107.95 153.67 0) (fields_autoplaced)
     (effects (font (size 1.27 1.27)) (justify left bottom))
@@
     (effects (font (size 1.27 1.27)) (justify left bottom))
   )
-  (label "DMX-RX" (at 24.13 135.89 0) (fields_autoplaced)
-    (effects (font (size 1.27 1.27)) (justify left bottom))
-  )
-  (label "ENC2-A" (at 107.95 120.65 0) (fields_autoplaced)
-    (effects (font (size 1.27 1.27)) (justify left bottom))
-  )
-  (label "MENU-LEFT" (at 182.88 118.11 180) (fields_autoplaced)
-    (effects (font (size 1.27 1.27)) (justify right bottom))
-  )
-  (label "DMX-TX" (at 24.13 144.78 0) (fields_autoplaced)
-    (effects (font (size 1.27 1.27)) (justify left bottom))
-  )
   (label "I2C-SCLK_{S}" (at 106.68 83.82 180) (fields_autoplaced)
     (effects (font (size 1.27 1.27)) (justify right bottom))
@@
     (effects (font (size 1.27 1.27)) (justify right bottom))
   )
+  (label "ENC2-A_{INT}" (at 107.95 120.65 0) (fields_autoplaced)
+    (effects (font (size 1.27 1.27)) (justify left bottom))
+  )
   (label "MIDI-OUT_{S}" (at 107.95 138.43 0) (fields_autoplaced)
     (effects (font (size 1.27 1.27)) (justify left bottom))
   )
-  (label "MENU-BACK" (at 182.88 113.03 180) (fields_autoplaced)
+  (label "MENU-ACT_{INT}" (at 182.88 123.19 180) (fields_autoplaced)
     (effects (font (size 1.27 1.27)) (justify right bottom))
   )
@@
     (effects (font (size 1.27 1.27)) (justify left bottom))
   )
-  (label "DMX-EN" (at 24.13 139.7 0) (fields_autoplaced)
-    (effects (font (size 1.27 1.27)) (justify left bottom))
-  )
   (label "SD-D0_{S}" (at 106.68 57.15 180) (fields_autoplaced)
     (effects (font (size 1.27 1.27)) (justify right bottom))
@@
     (effects (font (size 1.27 1.27)) (justify right bottom))
   )
+  (label "DMX-EN_{S}" (at 24.13 139.7 0) (fields_autoplaced)
+    (effects (font (size 1.27 1.27)) (justify left bottom))
+  )
   (label "MENU-LEFT_{INT}" (at 15.24 48.26 0) (fields_autoplaced)
     (effects (font (size 1.27 1.27)) (justify left bottom))
@@
   )
   (label "DMX-RX_{S}" (at 106.68 43.18 180) (fields_autoplaced)
-    (effects (font (size 1.27 1.27)) (justify right bottom))
-  )
-  (label "MENU-RIGHT" (at 182.88 125.73 180) (fields_autoplaced)
     (effects (font (size 1.27 1.27)) (justify right bottom))
   )
@@
       (effects (font (size 1.27 1.27)) (justify right))
     )
-    (pin "MENU-UP" output (at 162.56 115.57 0)
-      (effects (font (size 1.27 1.27)) (justify right))
-    )
-    (pin "MENU-ACT" output (at 162.56 123.19 0)
-      (effects (font (size 1.27 1.27)) (justify right))
-    )
-    (pin "MENU-LEFT" output (at 162.56 118.11 0)
-      (effects (font (size 1.27 1.27)) (justify right))
-    )
-    (pin "MENU-BACK" output (at 162.56 113.03 0)
-      (effects (font (size 1.27 1.27)) (justify right))
-    )
-    (pin "MENU-DOWN" output (at 162.56 120.65 0)
-      (effects (font (size 1.27 1.27)) (justify right))
-    )
-    (pin "MENU-RIGHT" output (at 162.56 125.73 0)
-      (effects (font (size 1.27 1.27)) (justify right))
-    )
+    (pin "MENU-UP_{INT}" output (at 162.56 115.57 0)
+      (effects (font (size 1.27 1.27)) (justify right))
+    )
+    (pin "MENU-ACT_{INT}" output (at 162.56 123.19 0)
+      (effects (font (size 1.27 1.27)) (justify right))
+    )
+    (pin "MENU-LEFT_{INT}" output (at 162.56 118.11 0)
+      (effects (font (size 1.27 1.27)) (justify right))
+    )
+    (pin "MENU-BACK_{INT}" output (at 162.56 113.03 0)
+      (effects (font (size 1.27 1.27)) (justify right))
+    )
+    (pin "MENU-DOWN_{INT}" output (at 162.56 120.65 0)
+      (effects (font (size 1.27 1.27)) (justify right))
+    )
+    (pin "MENU-RIGHT_{INT}" output (at 162.56 125.73 0)
+      (effects (font (size 1.27 1.27)) (justify right))
+    )

Commit message: PCB Lock REV11
Parts:
- added H1, H2, H3, H4: M2.5, MountingHole:MountingHole_2.7mm_M2.5_Pad_Via, symbol Mechanical:MountingHole_Pad
- JP1: footprint Jumper:SolderJumper-2_P1.3mm_Bridged2Bar_RoundedPad1.0x1.5mm -> Daxxn_Other:SMALL-JUMPER_0.2mm
Connections:
- net GND: now also H1.1, H2.1, H3.1, H4.1
Other:
- sheet INTERFACE CONNECTOR ports: added STRIP-PG; removed none
Changed lines of the file:
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@@
     (company "Daxxn Industries")
   )
+  (junction (at 105.41 179.07) (diameter 0) (color 0 0 0 0)
+  )
   (junction (at 74.93 134.62) (diameter 0) (color 0 0 0 0)
   )
@@
   (junction (at 53.34 118.11) (diameter 0) (color 0 0 0 0)
   )
+  (junction (at 113.03 179.07) (diameter 0) (color 0 0 0 0)
+  )
   (junction (at 45.72 124.46) (diameter 0) (color 0 0 0 0)
   )
+  (junction (at 109.22 179.07) (diameter 0) (color 0 0 0 0)
+  )
   (junction (at 36.83 139.7) (diameter 0) (color 0 0 0 0)
   )
@@
     (stroke (width 0.1) (type solid))
   )
+  (wire (pts (xy 162.56 151.13) (xy 182.88 151.13))
+    (stroke (width 0) (type default))
+  )
   (polyline (pts (xy 207.01 24.13) (xy 276.86 24.13))
     (stroke (width 0.1) (type solid))
@@
     (stroke (width 0) (type default))
   )
+  (wire (pts (xy 113.03 179.07) (xy 113.03 180.34))
+    (stroke (width 0) (type default))
+  )
   (wire (pts (xy 127 49.53) (xy 148.59 49.53))
     (stroke (width 0) (type default))
@@
     (stroke (width 0.1) (type solid))
   )
+  (wire (pts (xy 113.03 179.07) (xy 113.03 177.8))
+    (stroke (width 0) (type default))
+  )
   (wire (pts (xy 127 93.98) (xy 147.32 93.98))
     (stroke (width 0) (type default))
@@
     (stroke (width 0.1) (type solid))
   )
+  (wire (pts (xy 109.22 179.07) (xy 113.03 179.07))
+    (stroke (width 0) (type default))
+  )
   (polyline (pts (xy 207.01 41.91) (xy 276.86 41.91))
     (stroke (width 0.1) (type solid))
@@
     (stroke (width 0) (type default))
   )
+  (wire (pts (xy 101.6 177.8) (xy 101.6 179.07))
+    (stroke (width 0) (type default))
+  )
   (wire (pts (xy 127 57.15) (xy 148.59 57.15))
     (stroke (width 0) (type default))
@@
     (stroke (width 0) (type default))
   )
+  (wire (pts (xy 109.22 177.8) (xy 109.22 179.07))
+    (stroke (width 0) (type default))
+  )
   (wire (pts (xy 86.36 36.83) (xy 106.68 36.83))
     (stroke (width 0) (type default))
@@
     (stroke (width 0) (type default))
   )
-  (wire (pts (xy 162.56 152.4) (xy 182.88 152.4))
+  (wire (pts (xy 162.56 156.21) (xy 182.88 156.21))
     (stroke (width 0) (type default))
   )
@@
     (stroke (width 0) (type default))
   )
+  (wire (pts (xy 101.6 179.07) (xy 105.41 179.07))
+    (stroke (width 0) (type default))
+  )
   (wire (pts (xy 15.24 69.85) (xy 35.56 69.85))
     (stroke (width 0) (type default))
@@
     (stroke (width 0.1) (type solid))
   )
+  (wire (pts (xy 105.41 177.8) (xy 105.41 179.07))
+    (stroke (width 0) (type default))
+  )
   (polyline (pts (xy 193.04 54.102) (xy 198.12 54.102))
     (stroke (width 0.1) (type solid))
@@
   (polyline (pts (xy 193.04 66.802) (xy 198.12 66.802))
     (stroke (width 0.1) (type solid))
+  )
+  (wire (pts (xy 105.41 179.07) (xy 109.22 179.07))
+    (stroke (width 0) (type default))
   )
   (wire (pts (xy 107.95 123.19) (xy 128.27 123.19))
@@
     (effects (font (size 1.27 1.27)) (justify right bottom))
   )
-  (label "~{RESET}_{C}" (at 182.88 152.4 180) (fields_autoplaced)
+  (label "~{RESET}_{C}" (at 182.88 156.21 180) (fields_autoplaced)
     (effects (font (size 1.27 1.27)) (justify right bottom))
   )
@@
   )
   (label "MENU-UP_{INT}" (at 182.88 115.57 180) (fields_autoplaced)
+    (effects (font (size 1.27 1.27)) (justify right bottom))
+  )
+  (label "STRIP-PG" (at 182.88 151.13 180) (fields_autoplaced)
     (effects (font (size 1.27 1.27)) (justify right bottom))
   )
@@
     )
   )
+  (symbol (lib_id "Mechanical:MountingHole_Pad") (at 101.6 175.26 0) (unit 1)
+    (in_bom yes) (on_board yes) (dnp no)
+    (property "Reference" "H1" (at 101.6 171.45 0)
+      (effects (font (size 1.27 1.27)))
+    )
+    (property "Value" "M2.5" (at 99.06 173.99 0)
+      (effects (font (size 1.27 1.27)) (justify right))
+    )
+    (property "Footprint" "MountingHole:MountingHole_2.7mm_M2.5_Pad_Via" (at 101.6 175.26 0)
+      (effects (font (size 1.27 1.27)) hide)
+    )
+    (property "Datasheet" "~" (at 101.6 175.26 0)
+      (effects (font (size 1.27 1.27)) hide)
+    )
+    (property "Schematic" "" (at 101.6 175.26 0)
+      (effects (font (size 1.27 1.27)) hide)
+    )
+    (property "PartNumber" "" (at 101.6 175.26 0)
+      (effects (font (size 1.27 1.27)))
+    )
+    (property "SupplierPN" "" (at 101.6 175.26 0)
+      (effects (font (size 1.27 1.27)) hide)
+    )
+    (pin "1")
+    (instances
+      (project "LightDrum"
+        (path "/7f137461-fd46-4a4c-8db7-555d487fb3ca"
+          (reference "H1") (unit 1)
+        )
+      )
+    )
+  )
   (symbol (lib_id "power:GND") (at 53.34 153.67 0) (mirror y) (unit 1)
     (in_bom yes) (on_board yes) (dnp no)
@@
         (path "/7f137461-fd46-4a4c-8db7-555d487fb3ca"
           (reference "#PWR05") (unit 1)
+        )
+      )
+    )
+  )
+  (symbol (lib_id "power:GND") (at 113.03 180.34 0) (mirror y) (unit 1)
+    (in_bom yes) (on_board yes) (dnp no)
+    (property "Reference" "#PWR076" (at 113.03 186.69 0)
+      (effects (font (size 1.27 1.27)) hide)
+    )
+    (property "Value" "GND" (at 113.03 184.15 0)
+      (effects (font (size 1.27 1.27)))
+    )
+    (property "Footprint" "" (at 113.03 180.34 0)
+      (effects (font (size 1.27 1.27)) hide)
+    )
+    (property "Datasheet" "" (at 113.03 180.34 0)
+      (effects (font (size 1.27 1.27)) hide)
+    )
+    (pin "1")
+    (instances
+      (project "LightDrum"
+        (path "/7f137461-fd46-4a4c-8db7-555d487fb3ca"
+          (reference "#PWR076") (unit 1)
         )
       )
@@
     )
   )
+  (symbol (lib_id "Mechanical:MountingHole_Pad") (at 113.03 175.26 0) (unit 1)
+    (in_bom yes) (on_board yes) (dnp no)
+    (property "Reference" "H4" (at 113.03 171.45 0)
+      (effects (font (size 1.27 1.27)))
+    )
+    (property "Value" "M2.5" (at 113.03 170.815 0)
+      (effects (font (size 1.27 1.27)) hide)
+    )
+    (property "Footprint" "MountingHole:MountingHole_2.7mm_M2.5_Pad_Via" (at 113.03 175.26 0)
+      (effects (font (size 1.27 1.27)) hide)
+    )
+    (property "Datasheet" "~" (at 113.03 175.26 0)
+      (effects (font (size 1.27 1.27)) hide)
+    )
+    (property "Schematic" "" (at 113.03 175.26 0)
+      (effects (font (size 1.27 1.27)) hide)
+    )
+    (property "PartNumber" "" (at 113.03 175.26 0)
+      (effects (font (size 1.27 1.27)))
+    )
+    (property "SupplierPN" "" (at 113.03 175.26 0)
+      (effects (font (size 1.27 1.27)) hide)
+    )
+    (pin "1")
+    (instances
+      (project "LightDrum"
+        (path "/7f137461-fd46-4a4c-8db7-555d487fb3ca"
+          (reference "H4") (unit 1)
+        )
+      )
+    )
+  )
   (symbol (lib_id "Jumper:SolderJumper_2_Open") (at 74.93 144.78 90) (unit 1)
     (in_bom yes) (on_board yes) (dnp no)
@@
       (effects (font (size 1 1)) (justify right))
     )
-    (property "Footprint" "Jumper:SolderJumper-2_P1.3mm_Bridged2Bar_RoundedPad1.0x1.5mm" (at 74.93 144.78 0)
+    (property "Footprint" "Daxxn_Other:SMALL-JUMPER_0.2mm" (at 74.93 144.78 0)
       (effects (font (size 1.27 1.27)) hide)
     )
@@
     (property "SupplierPN" "~" (at 74.93 144.78 0)
       (effects (font (size 1.27 1.27)) hide)
+    )
+    (property "Schematic" "" (at 74.93 144.78 0)
+      (effects (font (size 1.27 1.27)) hide)
+    )
+    (property "PartNumber" "" (at 74.93 144.78 0)
+      (effects (font (size 1.27 1.27)))
     )
     (pin "1")
@@
     )
   )
+  (symbol (lib_id "Mechanical:MountingHole_Pad") (at 109.22 175.26 0) (unit 1)
+    (in_bom yes) (on_board yes) (dnp no)
+    (property "Reference" "H3" (at 109.22 171.45 0)
+      (effects (font (size 1.27 1.27)))
+    )
+    (property "Value" "M2.5" (at 109.22 170.815 0)
+      (effects (font (size 1.27 1.27)) hide)
+    )
+    (property "Footprint" "MountingHole:MountingHole_2.7mm_M2.5_Pad_Via" (at 109.22 175.26 0)
+      (effects (font (size 1.27 1.27)) hide)
+    )
+    (property "Datasheet" "~" (at 109.22 175.26 0)
+      (effects (font (size 1.27 1.27)) hide)
+    )
+    (property "Schematic" "" (at 109.22 175.26 0)
+      (effects (font (size 1.27 1.27)) hide)
+    )
+    (property "PartNumber" "" (at 109.22 175.26 0)
+      (effects (font (size 1.27 1.27)))
+    )
+    (property "SupplierPN" "" (at 109.22 175.26 0)
+      (effects (font (size 1.27 1.27)) hide)
+    )
+    (pin "1")
+    (instances
+      (project "LightDrum"
+        (path "/7f137461-fd46-4a4c-8db7-555d487fb3ca"
+          (reference "H3") (unit 1)
+        )
+      )
+    )
+  )
+  (symbol (lib_id "Mechanical:MountingHole_Pad") (at 105.41 175.26 0) (unit 1)
+    (in_bom yes) (on_board yes) (dnp no)
+    (property "Reference" "H2" (at 105.41 171.45 0)
+      (effects (font (size 1.27 1.27)))
+    )
+    (property "Value" "M2.5" (at 105.41 170.815 0)
+      (effects (font (size 1.27 1.27)) hide)
+    )
+    (property "Footprint" "MountingHole:MountingHole_2.7mm_M2.5_Pad_Via" (at 105.41 175.26 0)
+      (effects (font (size 1.27 1.27)) hide)
+    )
+    (property "Datasheet" "~" (at 105.41 175.26 0)
+      (effects (font (size 1.27 1.27)) hide)
+    )
+    (property "Schematic" "" (at 105.41 175.26 0)
+      (effects (font (size 1.27 1.27)) hide)
+    )
+    (property "PartNumber" "" (at 105.41 175.26 0)
+      (effects (font (size 1.27 1.27)))
+    )
+    (property "SupplierPN" "" (at 105.41 175.26 0)
+      (effects (font (size 1.27 1.27)) hide)
+    )
+    (pin "1")
+    (instances
+      (project "LightDrum"
+        (path "/7f137461-fd46-4a4c-8db7-555d487fb3ca"
+          (reference "H2") (unit 1)
+        )
+      )
+    )
+  )
   (sheet (at 148.59 41.91) (size 26.67 17.78)
     (stroke (width 0.1524) (type solid))
@@
       (effects (font (size 1.27 1.27)) (justify left))
     )
-    (pin "~{RESET}_{C}" input (at 162.56 152.4 0)
+    (pin "~{RESET}_{C}" input (at 162.56 156.21 0)
       (effects (font (size 1.27 1.27)) (justify right))
     )
@@
       (effects (font (size 1.27 1.27)) (justify left))
     )
+    (pin "STRIP-PG" input (at 162.56 151.13 0)
+      (effects (font (size 1.27 1.27)) (justify right))
+    )
     (instances
