File: LightDrumInterface/LightDrumInterface.kicad_pcb (KiCad board)
At the start: 2 copper layers, 108 x 83 mm, 61 parts, among them J1 Conn_01x04_Male, J2 DEBUG-CONN, J3 Conn_01x04_Male, J4 PWR-CONN, J6 0541323662, SW1 RESET-SW, U1 STP16CP05, U101 LTC4054ES5-4.2, U2 TPL0401B-10-Q1, U3 74AUP2G04, U4 PC817

Commit message: interface layout completed - REV6
Parts:
- removed BAT101: 12mm COIN, Battery:BatteryHolder_Keystone_3000_1x12mm
- removed C101: 100nF, Capacitor_SMD:C_0603_1608Metric
- removed the G*** at (-70.0, 46.5)
- removed the G*** at (-72.5, 46.5)
- removed J2: DEBUG-CONN, Connector_JST:JST_XH_B4B-XH-A_1x04_P2.50mm_Vertical
- removed R101: 1.2K, Resistor_SMD:R_0603_1608Metric
- removed S-ACT1, S-DWN1, S-LFT1, S-RGT1, S-UP1: ILS, Daxxn_Switches:ILS-TB
- removed U101: LTC4054ES5-4.2, Package_TO_SOT_SMD:TSOT-23-5
- removed kibuzzard-62EEA0C0: G***, kibuzzard-62EEA0C0
- removed kibuzzard-62EEA0FE: G***, kibuzzard-62EEA0FE
- added D-BK1: RED, LED_SMD:LED_0805_2012Metric, F.Cu at (-5.50, 25.4)
- added D-BK2: RED, LED_SMD:LED_0805_2012Metric, F.Cu at (-5.50, 39.4)
- added D-BK3: RED, LED_SMD:LED_0805_2012Metric, F.Cu at (-24.5, 39.4)
- added D-BK4: RED, LED_SMD:LED_0805_2012Metric, F.Cu at (-24.5, 25.4)
- added D-MB1: RED, LED_SMD:LED_0805_2012Metric, F.Cu at (-33.3, 32.6)
- added D-MD1: RED, LED_SMD:LED_0805_2012Metric, F.Cu at (-15.0, 40.3)
- added D-ML1: RED, LED_SMD:LED_0805_2012Metric, F.Cu at (-25.0, 32.4)
- added D-MR1: RED, LED_SMD:LED_0805_2012Metric, F.Cu at (-5.00, 32.4)
- added D-MU1: RED, LED_SMD:LED_0805_2012Metric, F.Cu at (-15.0, 24.4)
- added D-VDD1: YELLOW, LED_SMD:LED_0805_2012Metric, F.Cu at (13.0, -29.5)
- added G***: LOGO, Daxxn_Logos_Art:LightDrum_Logo_SLK_15mm, F.Cu at (31.5, -33.0)
- added G***: LOGO, Daxxn_Logos_Art:LightDrum_Logo_FCu_15mm, F.Cu at (31.5, -33.0)
- added J5: MIDI-OUT, Connector_PinHeader_2.54mm:PinHeader_1x04_P2.54mm_Vertical, B.Cu at (36.0, -8.20)
- added Q1: NX6008NBKWX, Package_TO_SOT_SMD:SOT-323_SC-70, F.Cu at (17.0, -15.0)
- added Q2: NX6008NBKWX, Package_TO_SOT_SMD:SOT-323_SC-70, F.Cu at (1.00, -15.0)
- added Q3: NX6008NBKWX, Package_TO_SOT_SMD:SOT-323_SC-70, F.Cu at (-4.00, -15.0)
- added Q4: NX6008NBKWX, Package_TO_SOT_SMD:SOT-323_SC-70, F.Cu at (22.0, -15.0)
- added R1: 100, Resistor_SMD:R_0805_2012Metric, F.Cu at (17.0, -18.5)
- added R16: 560Ω, Resistor_SMD:R_0805_2012Metric, F.Cu at (-14.9, -2.90)
- added R18: 10KΩ, Resistor_SMD:R_0805_2012Metric, F.Cu at (26.0, 22.3)
- added R19: 220Ω, Resistor_SMD:R_0805_2012Metric, F.Cu at (29.7, 10.7)
- added R20: 10KΩ, Resistor_SMD:R_0805_2012Metric, F.Cu at (19.9, 16.0)
- added R21: 10KΩ, Resistor_SMD:R_0805_2012Metric, F.Cu at (13.0, 22.3)
- added R22: 10KΩ, Resistor_SMD:R_0805_2012Metric, F.Cu at (7.00, 22.3)
- added R23: 220Ω, Resistor_SMD:R_0805_2012Metric, F.Cu at (39.3, -9.20)
- added R24: 220Ω, Resistor_SMD:R_0805_2012Metric, F.Cu at (32.3, -13.3)
- added SN1: JS5208, Daxxn_Switches:JS5208, F.Cu at (-15.0, 32.4)
- C1, JP1: moved to B.Cu
- C3: value 100nF -> 1uF
- C9: value 1uF -> 100nF; moved to F.Cu
- DS1: value NX4024T032 -> NX4024K032; footprint Daxxn_Displays:NX4024T032_10mm -> Daxxn_Displays:NX4024K032-RA-S04B
- ENC1, ENC2: footprint Daxxn_Switches:PEC12R -> Daxxn_Switches:PEC11R
- J1: value Conn_01x04_Male -> MIDI-IN; moved to B.Cu
- J3: value Conn_01x04_Male -> DEBUG-CONN; footprint Connector_PinHeader_2.54mm:PinHeader_1x04_P2.54mm_Vertical -> Connector_JST:JST_XH_B4B-XH-A_1x04_P2.50mm_Vertical; moved to B.Cu
- R10, R11, R12, R9: value 10KΩ -> 100; moved to B.Cu
- R13: value 220Ω -> 1.3K
- R14: value 220Ω -> 560
- R15: value 220Ω -> 4.7K
- R2: value 560Ω -> 550
- R3: value 330Ω -> 620
- R4: value 330Ω -> 100
- R5: value 470Ω -> 10K
- R6: value 330Ω -> 10K
- R7: value 3KΩ -> 10K
- R8: value 5.6KΩ -> 10K
- S-BCK1: value ILS -> M-BACK; footprint Daxxn_Switches:ILS-TB -> Daxxn_Switches:TL3365AF180QG
- U3: value 74AUP2G04 -> PC817; footprint Package_TO_SOT_SMD:SOT-363_SC-70-6 -> Package_DIP:DIP-4_W7.62mm
- U4: value PC817 -> 74AUP2G04; footprint Package_DIP:DIP-4_W7.62mm -> Package_TO_SOT_SMD:SOT-363_SC-70-6
- moved SW1 90.9 mm to (-51.0, 16.0), turned to 90 degrees
- moved ENC1 88.2 mm to (29.0, 32.7), turned to 180 degrees
- moved C5 79.1 mm to (30.0, 22.3), turned to 90 degrees
- moved C6 74.8 mm to (28.0, 22.3), turned to -90 degrees
- moved C9 68.6 mm to (32.0, -15.2), turned to 0 degrees
- moved ENC2 62.5 mm to (10.0, 32.6), turned to 180 degrees
- moved J3 62.3 mm to (-41.5, 3.75), turned to 90 degrees
- moved C7 54.0 mm to (11.0, 22.3), turned to 90 degrees
- moved C8 50.7 mm to (9.00, 22.3), turned to -90 degrees
- moved R10 49.0 mm to (-2.10, 21.0), turned to 90 degrees
- moved R9 48.7 mm to (-4.10, 21.0), turned to 90 degrees
- moved R7 42.4 mm to (-4.00, -12.3), turned to 0 degrees
- moved J1 42.1 mm to (36.0, 15.8), turned to 0 degrees
- moved D1 37.4 mm to (32.9, 12.0), turned to 90 degrees
- moved R11 36.7 mm to (-6.10, 21.0), turned to 90 degrees
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Connections:
- C3 pad 1: VDD -> VCC
- C4 pad 1: VCC -> VDD
- C9 pad 1: VDD -> VCC
- D-AUDIO-SEL1 pad 2: /AUDIO-RELAY -> VCC
- D-DBG1 pad 2: VDD -> VCC
- D-STA1 pad 2: VDD -> VCC
- D-STRIP-EN1 pad 2: VDD -> VCC
- D-VCC1 pad 2: VDD -> VCC
- DA1 pad 1: VDD -> VCC
- DA1 pad 10: VDD -> VCC
- DA1 pad 2: VDD -> VCC
- DA1 pad 3: VDD -> VCC
- DA1 pad 4: VDD -> VCC
- DA1 pad 5: VDD -> VCC
- DA1 pad 6: VDD -> VCC
- DA1 pad 7: VDD -> VCC
- DA1 pad 8: VDD -> VCC
- DA1 pad 9: VDD -> VCC
- J3 pad 2: Net-(J3-Pad2) -> /I2C-SCLK
- J3 pad 3: Net-(J3-Pad3) -> /I2C-SDA
- J6 pad 1: /AUDIO-RELAY -> VDD
- J6 pad 10: /ENC1-A -> /ENC1-SW
- J6 pad 11: I2C-SDA -> /ENC2-A
- J6 pad 12: /ENC1-B -> /ENC2-B
- J6 pad 14: /VBAT -> /I2C-SDA
- J6 pad 15: /GRAPH-~{OE} -> /ENC2-SW
- J6 pad 16: /MENU-UP -> /SCR-TX
- J6 pad 17: /GRAPH-SDI -> /I2C-SCLK
- J6 pad 18: /MENU-ACT -> /SCR-RX
- J6 pad 19: /GRAPH-CLK -> /MENU-RIGHT
- J6 pad 2: Vdrive -> /MIDI-OUT
- J6 pad 20: /MENU-DOWN -> /MENU-ACT
- J6 pad 21: /GRAPH-LE -> /MENU-BACK
- J6 pad 22: /MENU-LEFT -> /MENU-UP
- J6 pad 23: /CHARGE-STATUS -> /GRAPH-LE
- J6 pad 24: /MENU-BACK -> /MENU-LEFT
- J6 pad 25: /MIDI-IN -> /GRAPH-~{OE}
- J6 pad 26: /MENU-RIGHT -> /MENU-DOWN
- J6 pad 27: /MIDI-OUT -> /ENC1-B
- J6 pad 3: /ENC1-SW -> GND
- J6 pad 31: /SCR-TX -> /DIAG-STATUS
- J6 pad 32: /DIAG-STATUS -> /DIAG-DEBUG
- J6 pad 33: /SCR-RX -> /AUDIO-SRC-IND
- J6 pad 34: /DIAG-DEBUG -> GND
- J6 pad 36: ~{RESET} -> Vdrive
- J6 pad 4: VDD -> /~{RESET}
- J6 pad 5: /ENC2-SW -> /MIDI-IN
- J6 pad 6: /ENC2-B -> /GRAPH-SDI
- J6 pad 8: /ENC2-A -> /GRAPH-CLK
- J6 pad 9: I2C-SCLK -> /ENC1-A
- R10 pad 1: VDD -> Net-(D-BK2-Pad1)
- R10 pad 2: /ENC1-B -> /NAV-BACKLIGHT
- R11 pad 1: /ENC2-A -> Net-(D-BK3-Pad1)
- R11 pad 2: VDD -> /NAV-BACKLIGHT
- R12 pad 1: VDD -> Net-(D-BK4-Pad1)
- R12 pad 2: /ENC2-B -> /NAV-BACKLIGHT
- R13 pad 1: Net-(D1-Pad2) -> Net-(D-VDD1-Pad1)
- R13 pad 2: Net-(R13-Pad2) -> GND
- R14 pad 1: Net-(J3-Pad2) -> Net-(D-VCC1-Pad1)
- R14 pad 2: VCC -> GND
- R15 pad 1: Net-(J3-Pad3) -> Net-(D-VDRIVE1-Pad1)
- R15 pad 2: Net-(R15-Pad2) -> GND
- R17 pad 1: /MIDI-IN -> /ENC1-A
- R17 pad 2: VCC -> VDD
- R2 pad 1: Net-(JP1-Pad1) -> Net-(D-STA1-Pad1)
- R2 pad 2: GND -> Net-(Q2-Pad3)
- R3 pad 1: Net-(D-AUDIO-SEL1-Pad1) -> Net-(D-DBG1-Pad1)
- R3 pad 2: GND -> Net-(Q3-Pad3)
- R4 pad 1: Net-(D-STRIP-EN1-Pad1) -> Net-(D-AUDIO-SEL1-Pad1)
- R4 pad 2: /STRIP-PWR -> Net-(Q4-Pad3)
- R5 pad 1: Net-(D-STA1-Pad1) -> /STRIP-PWR
- R5 pad 2: /DIAG-STATUS -> GND
- R6 pad 1: Net-(D-DBG1-Pad1) -> /DIAG-STATUS
- R6 pad 2: /DIAG-DEBUG -> GND
- R7 pad 1: Net-(D-VCC1-Pad1) -> /DIAG-DEBUG
- R8 pad 1: Net-(D-VDRIVE1-Pad1) -> /AUDIO-SRC-IND
- R9 pad 1: /ENC1-A -> Net-(D-BK1-Pad1)
- R9 pad 2: VDD -> /NAV-BACKLIGHT
- S-BCK1 pad 1: /MENU-BACK -> GND
- S-BCK1 pad 2: (no net) -> /MENU-BACK
- SW1 pad 2: ~{RESET} -> /~{RESET}
- U1 pad 19: Net-(S-BCK1-Pad6) -> Net-(U1-Pad19)
- U1 pad 20: Net-(S-RGT1-Pad6) -> /NAV-BACKLIGHT
- U2 pad 3: I2C-SCLK -> /I2C-SCLK
- U2 pad 4: I2C-SDA -> /I2C-SDA
- U3 pad 1: /MIDI-OUT -> Net-(D1-Pad1)
- U3 pad 2: GND -> Net-(R19-Pad2)
- U3 pad 3: Net-(U3-Pad3) -> GND
- U3 pad 4: Net-(R15-Pad2) -> /MIDI-IN
- U4 pad 1: Net-(D1-Pad1) -> /MIDI-OUT
- U4 pad 2: Net-(R13-Pad2) -> GND
- U4 pad 3: GND -> Net-(U4-Pad3)
- U4 pad 4: /MIDI-IN -> Net-(R24-Pad2)
Routing:
- net VCC: track 0.00 -> 415.4 mm, vias 0 -> 15
- net VDD: track 0.00 -> 241.0 mm, vias 0 -> 11
- net Vdrive: track 0.00 -> 149.9 mm, vias 0 -> 1
- net /AUDIO-SRC-IND: track 0.00 -> 92.8 mm, vias 0 -> 3
- net Net-(U1-Pad18): track 0.00 -> 90.8 mm, vias 0 -> 6
- net /ENC1-A: track 0.00 -> 86.2 mm, vias 0 -> 1
- net /ENC1-B: track 0.00 -> 85.0 mm, vias 0 -> 1
- net /MIDI-OUT: track 0.00 -> 81.7 mm, vias 0 -> 3
- net /ENC1-SW: track 0.00 -> 81.6 mm, vias 0 -> 1
- net /STRIP-PWR: track 0.00 -> 79.9 mm, vias 0 -> 1
- net /DIAG-DEBUG: track 0.00 -> 73.9 mm, vias 0 -> 1
- net /NAV-BACKLIGHT: track 0.00 -> 73.9 mm, vias 0 -> 5
- net /I2C-SDA: track 0.00 -> 71.3 mm, vias 0 -> 1
- net /DIAG-STATUS: track 0.00 -> 70.6 mm, vias 0 -> 1
- net Net-(U1-Pad15): track 0.00 -> 68.8 mm, vias 0 -> 6
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- added copper zone on B.Cu, net GND
- added copper zone on F.Cu, net GND
Other:
- board text added: "AUDIO GAIN"
- board text added: "AUDIO SOURCE"
- board text added: "MIDI IN"
- board text added: "MIDI OUT"
- board text added: "REV9"
- board text added: "VDD"
- board text removed: "AUDIO SELECT"
- board text removed: "DEBUG"
- board text removed: "DOWN"
- board text removed: "ENTER"
- board text removed: "EXTERN MIDI"
- board text removed: "LEFT"
- board text removed: "REV8"
- board text removed: "RIGHT"
- board text removed: "UP"

Commit message: interface layout completed - REV6
Parts:
- moved C1 98.5 mm to (97.8, 66.0)
- moved C2 98.5 mm to (62.5, 53.0)
- moved C3 98.5 mm to (65.5, 27.8)
- moved C4 98.5 mm to (61.1, 63.1)
- moved C5 98.5 mm to (103.2, 88.3)
- moved C6 98.5 mm to (101.2, 88.3)
- moved C7 98.5 mm to (84.2, 88.3)
- moved C8 98.5 mm to (82.2, 88.3)
- moved C9 98.5 mm to (105.2, 50.8)
- moved D-AUDIO-SEL1 98.5 mm to (94.2, 28.0)
- moved D-BK1 98.5 mm to (67.7, 91.4)
- moved D-BK2 98.5 mm to (67.7, 105.4)
- moved D-BK3 98.5 mm to (48.6, 105.4)
- moved D-BK4 98.5 mm to (48.6, 91.4)
- moved D-DBG1 98.5 mm to (68.2, 28.0)
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